File: Board_STM32F103C8T6/STM32F103C8T6/STM32F103C8T6.kicad_pcb (KiCad board)
At the start: 2 copper layers, 96 x 96 mm, 104 parts, among them J301 BOOT, J401 BATTERY, J402 I2C, J403 H2O, J404 USB_B_Micro, J405 SWD, J406 USART1, J407 CIRCUIT_SENSOR, J408 BLUETOOTH, J409 RPM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

Commit message: Updated board design
work in progress
Parts:
- added C703: 10u, Capacitor_SMD:C_1206_3216Metric_Pad1.33x1.80mm_HandSolder, F.Cu at (85.5, 58.0)
- added H307: MountingHole, MyFootprints:JLCPCB-Tooling-Hole, F.Cu at (94.5, 122.5)
- added H308: MountingHole, MyFootprints:JLCPCB-Tooling-Hole, F.Cu at (96.7, 122.5)
- added H309: MountingHole, MyFootprints:JLCPCB-Tooling-Hole, F.Cu at (98.8, 122.5)
- added J801: Conn_Coaxial, MyFootprints:BWIPX-1-001E, F.Cu at (151.5, 34.5)
- C701: footprint Capacitor_SMD:C_0603_1608Metric_Pad1.08x0.95mm_HandSolder -> Capacitor_SMD:C_1206_3216Metric_Pad1.33x1.80mm_HandSolder
- C702: footprint Capacitor_SMD:C_0603_1608Metric_Pad1.08x0.95mm_HandSolder -> Capacitor_SMD:C_1210_3225Metric_Pad1.33x2.70mm_HandSolder
- FB201: footprint Inductor_SMD:L_0805_2012Metric -> Inductor_SMD:L_1206_3216Metric_Pad1.22x1.90mm_HandSolder
- L301, L801: footprint Inductor_SMD:L_0402_1005Metric -> Inductor_SMD:L_0402_1005Metric_Pad0.77x0.64mm_HandSolder
- Q301: value VP0610T -> AO3401A
- R701, R702, R706: footprint Resistor_SMD:R_0603_1608Metric_Pad0.98x0.95mm_HandSolder -> Resistor_SMD:R_1206_3216Metric_Pad1.30x1.75mm_HandSolder
- R703, R704, R705: footprint Resistor_SMD:R_0603_1608Metric_Pad0.98x0.95mm_HandSolder -> Resistor_SMD:R_1210_3225Metric_Pad1.30x2.65mm_HandSolder
- Y301: footprint Crystal:Crystal_SMD_5032-2Pin_5.0x3.2mm -> Crystal:Crystal_SMD_5032-2Pin_5.0x3.2mm_HandSoldering
- moved D701 161.4 mm to (130.0, 118.0), turned to 180 degrees
- moved C702 158.3 mm to (132.0, 112.0), turned to 270 degrees
- moved R312 151.6 mm to (89.5, 97.0)
- moved R704 151.3 mm to (128.0, 112.0), turned to 270 degrees
- moved D704 150.6 mm to (119.0, 109.5), turned to 270 degrees
- moved R705 148.5 mm to (129.0, 102.5), turned to 270 degrees
- moved C311 147.1 mm to (110.1, 82.0)
- moved D703 145.3 mm to (123.5, 105.0), turned to 270 degrees
- moved D702 143.4 mm to (136.5, 111.5), turned to 270 degrees
- moved R313 143.3 mm to (147.3, 82.5), turned to 270 degrees
- moved R317 140.7 mm to (78.5, 69.0), turned to 270 degrees
- moved R304 138.6 mm to (161.5, 75.0), turned to 270 degrees
- moved R703 137.4 mm to (136.5, 104.0), turned to 270 degrees
- moved R311 135.8 mm to (89.5, 93.5)
- moved L301 135.8 mm to (116.5, 77.5), turned to 90 degrees
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Routing:
- net LSE_IN: track 0.00 -> 18.5 mm
- net HSE_IN: track 0.00 -> 14.2 mm
- net LSE_OUT: track 0.00 -> 12.4 mm
- net Net-(C311-Pad1): track 0.00 -> 11.8 mm
- net HSE_OUT: track 0.00 -> 9.59 mm
- net GND: track 0.00 -> 6.45 mm, vias 0 -> 4
- net Net-(C312-Pad1): track 0.00 -> 4.89 mm
- added copper zone on In2.Cu, net +3V3
- added copper zone on B.Cu, net GND
- added copper zone on F.Cu, net GND
- added copper zone on In1.Cu, net GND
- added copper zone on B.Cu, net GND1
- added copper zone on In1.Cu, net GND1
- added copper zone on In2.Cu, net GND1
Other:
- copper layers 2 -> 4
- net class Default: clearance 0.2 -> 0.1
- rule trace_clearance: 0.2 -> 0.1
- rule via_min_drill: 0.3 -> 0.4
- rule via_min_size: 0.4 -> 0.5

Commit message: Improved PCB layout
Parts:
- added C402: 47p, Capacitor_SMD:C_0402_1005Metric_Pad0.74x0.62mm_HandSolder, F.Cu at (129.8, 50.9)
- added C403: 47p, Capacitor_SMD:C_0402_1005Metric_Pad0.74x0.62mm_HandSolder, F.Cu at (123.0, 46.8)
- added R401: 22, Resistor_SMD:R_0402_1005Metric_Pad0.72x0.64mm_HandSolder, F.Cu at (127.5, 50.2)
- added R402: 22, Resistor_SMD:R_0402_1005Metric_Pad0.72x0.64mm_HandSolder, F.Cu at (119.9, 46.8)
- C401: value 10u -> 100n
- Q301: value AO3401A -> BSS123
- moved H308 75.2 mm to (86.5, 48.0)
- moved H309 61.7 mm to (160.0, 114.5)
- moved H307 6.00 mm to (88.5, 122.5)
- moved R319 4.30 mm to (119.9, 48.8), turned to 180 degrees
- moved J410 2.59 mm to (75.0, 88.0), turned to 0 degrees
- moved C303 1.12 mm to (122.0, 67.0), turned to 0 degrees
- moved C305 1.12 mm to (127.0, 80.0), turned to 180 degrees
- moved Q301 0.96 mm to (124.1, 52.5)
- moved C501 0.76 mm to (139.5, 49.7)
- moved C503 0.76 mm to (139.5, 47.7)
- moved C601 0.74 mm to (114.5, 49.7)
- moved C602 0.74 mm to (114.5, 51.7)
- moved C304 0.71 mm to (131.0, 70.5), turned to 270 degrees
- moved R320 0.56 mm to (122.4, 56.0), turned to 0 degrees
- moved R303 0.40 mm to (161.5, 70.9)
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Connections:
- C401 pad 1: +5V -> +3V3
- Q301 pad 2: +3V3 -> GND
- Q301 pad 3: Net-(Q301-Pad3) -> USB_D+
- R319 pad 2: Net-(Q301-Pad3) -> +3V3
- R320 pad 1: GND -> +3V3
- U401 pad 4: USB_D+ -> Net-(R402-Pad2)
- U401 pad 5: +5V -> +3V3
- U401 pad 6: USB_D- -> Net-(R401-Pad1)
Routing:
- net +3V3: track 0.00 -> 151.7 mm, vias 0 -> 40
- net TRACK_SENSOR: track 0.00 -> 105.1 mm, vias 0 -> 1
- net USART2_TX: track 0.00 -> 97.1 mm, vias 0 -> 1
- net USART2_RX: track 0.00 -> 94.2 mm, vias 0 -> 1
- net GPS_ONOFF: track 0.00 -> 82.9 mm, vias 0 -> 2
- net GPS_PPS: track 0.00 -> 81.8 mm, vias 0 -> 2
- net +5V: track 0.00 -> 72.3 mm, vias 0 -> 2
- net NRST: track 0.00 -> 70.0 mm, vias 0 -> 2
- net BOOT0: track 0.00 -> 67.4 mm, vias 0 -> 2
- net SWO: track 0.00 -> 61.9 mm, vias 0 -> 1
- net GND: track 6.45 -> 65.7 mm, vias 4 -> 94
- net SWCLK: track 0.00 -> 58.9 mm
- net H2O_NTC+: track 0.00 -> 54.9 mm, vias 0 -> 1
- net 12C1_SDA: track 0.00 -> 50.6 mm, vias 0 -> 3
- net SWDIO: track 0.00 -> 47.4 mm
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Other:
- net class Default: clearance 0.1 -> 0.2
- rule trace_clearance: 0.1 -> 0.2
- board text added: "+"
- board text added: "+BATT"
- board text added: "-"
- board text added: "-BATT"
- board text added: "BOOT"
- board text added: "H2O"
- board text added: "JLCJLCJLCJLC"
- board text added: "POWER"
- board text added: "RPM"
- board text added: "RX1"
- board text added: "RX2"
- board text added: "SCL1"
- board text added: "SDA1"
- board text added: "STATUS"
- board text added: "STMF103 BADIBOARD || REV1"
- board text added: "TRACK"
- board text added: "TX1"
- board text added: "TX2"
