File: Board_STM32F103C8T6/STM32F103C8T6/STM32F103C8T6.kicad_pcb (KiCad board)
At the start: 4 copper layers, 96 x 96 mm, 115 parts, among them J301 BOOT, J401 BATTERY, J402 I2C, J403 H2O, J404 USB_C_Receptacle_USB2.0, J405 SWD, J406 USART1, J407 CIRCUIT_SENSOR, J408 BLUETOOTH, J409 RPM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

Commit message: Updated version from 5.1.9 to 6.0.5 (#7)
Other:
- net class Default removed
