File: Board_STM32F103C8T6/STM32F103C8T6/_autosave-STM32F103C8T6.kicad_pcb (KiCad board)
At the start: 4 copper layers, 96 x 96 mm, 113 parts, among them J301 BOOT, J401 BATTERY, J402 I2C, J403 H2O, J404 USB_B_Micro, J405 SWD, J406 USART1, J407 CIRCUIT_SENSOR, J408 BLUETOOTH, J409 RPM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

Commit message: added files to product pcb
Parts:
- C702: value 250n -> 220n
- R703: value 4,7K -> 4k7
- U201: value LD1117S33TR_SOT223 -> LD1117S33TR
