File: Board_STM32F103C8T6/STM32F103C8T6/IMU.sch (KiCad schematic (older format))
At the start: 6 parts, among them U501 MPU-6050

Commit message: Changed Crystals
Parts:
- C501: value 10u -> 10uF; Mouser (none) -> 581-0402ZD106MAT2A
- C502, C503, C504: value 100n -> 0.1uF; Mouser (none) -> 581-0402YD104K
- C505: value 2n2 -> 2200pF; Mouser (none) -> 581-0402YC222J4T2A
Changed lines of the file:
@@
 P 5050 2050
 F 0 "C501" H 5100 2100 50  0000 L CNN
-F 1 "10u" H 5100 2000 50  0000 L CNN
+F 1 "10uF" H 5100 2000 50  0000 L CNN
 F 2 "Capacitor_SMD:C_0402_1005Metric_Pad0.74x0.62mm_HandSolder" H 5050 2050 50  0001 C CNN
 F 3 "~" H 5050 2050 50  0001 C CNN
 F 4 "C15525" H 5050 2050 50  0001 C CNN "LCSC Part #"
+F 5 "581-0402ZD106MAT2A" H 5050 2050 50  0001 C CNN "Mouser"
 	1    5050 2050
 	1    0    0    -1
@@
 P 5350 2050
 F 0 "C502" H 5400 2100 50  0000 L CNN
-F 1 "100n" H 5400 2000 50  0000 L CNN
+F 1 "0.1uF" H 5400 2000 50  0000 L CNN
 F 2 "Capacitor_SMD:C_0402_1005Metric_Pad0.74x0.62mm_HandSolder" H 5350 2050 50  0001 C CNN
 F 3 "~" H 5350 2050 50  0001 C CNN
 F 4 "C1525" H 5350 2050 50  0001 C CNN "LCSC Part #"
+F 5 "581-0402YD104K" H 5350 2050 50  0001 C CNN "Mouser"
 	1    5350 2050
 	1    0    0    -1
@@
 P 5700 2050
 F 0 "C503" H 5750 2100 50  0000 L CNN
-F 1 "100n" H 5750 2000 50  0000 L CNN
+F 1 "0.1uF" H 5750 2000 50  0000 L CNN
 F 2 "Capacitor_SMD:C_0402_1005Metric_Pad0.74x0.62mm_HandSolder" H 5700 2050 50  0001 C CNN
 F 3 "~" H 5700 2050 50  0001 C CNN
 F 4 "C1525" H 5700 2050 50  0001 C CNN "LCSC Part #"
+F 5 "581-0402YD104K" H 5700 2050 50  0001 C CNN "Mouser"
 	1    5700 2050
 	1    0    0    -1
@@
 P 6200 3950
 F 0 "C504" H 6250 4000 50  0000 L CNN
-F 1 "100n" H 6250 3900 50  0000 L CNN
+F 1 "0.1uF" H 6250 3900 50  0000 L CNN
 F 2 "Capacitor_SMD:C_0402_1005Metric_Pad0.74x0.62mm_HandSolder" H 6200 3950 50  0001 C CNN
 F 3 "~" H 6200 3950 50  0001 C CNN
 F 4 "C1525" H 6200 3950 50  0001 C CNN "LCSC Part #"
+F 5 "581-0402YD104K" H 6200 3950 50  0001 C CNN "Mouser"
 	1    6200 3950
 	1    0    0    -1
@@
 P 6550 3950
 F 0 "C505" H 6600 4000 50  0000 L CNN
-F 1 "2n2" H 6600 3900 50  0000 L CNN
+F 1 "2200pF" H 6600 3900 50  0000 L CNN
 F 2 "Capacitor_SMD:C_0402_1005Metric_Pad0.74x0.62mm_HandSolder" H 6550 3950 50  0001 C CNN
 F 3 "~" H 6550 3950 50  0001 C CNN
 F 4 "C1531" H 6550 3950 50  0001 C CNN "LCSC Part #"
+F 5 "581-0402YC222J4T2A" H 6550 3950 50  0001 C CNN "Mouser"
 	1    6550 3950
 	1    0    0    -1
