File: Board_STM32F103C8T6/STM32F103C8T6/BLUETOOTH.sch (KiCad schematic (older format))
At the start: 7 parts, among them U601 HM-19_Module

Commit message: Updated board design
work in progress
Parts:
- U601: value HM-19_Module -> HM-19
Changed lines of the file:
@@
 P 6000 3650
 F 0 "U601" H 6350 4200 60  0000 C CNN
-F 1 "HM-19_Module" H 6400 3150 60  0000 C CNN
+F 1 "HM-19" H 6400 3150 60  0000 C CNN
 F 2 "Charleslabs_Parts:HM-11_Module" H 6000 3100 60  0001 C CNN
 F 3 "" H 6000 1800 60  0000 C CNN

Commit message: Changed Crystals
Parts:
- C601: value 10u -> 10uF; Mouser (none) -> 581-0402ZD106MAT2A
- C602: value 100n -> 0.1uF; Mouser (none) -> 581-0402YD104K
- D601: Mouser (none) -> 710-150060RS75020
- R601, R602: value 1k -> 1kΩ
- R603: value 1k5 -> 1.5kΩ
Changed lines of the file:
@@
 AR Path="/60860E11/60864A89" Ref="C601"  Part="1"
 F 0 "C601" H 5850 2200 50  0000 L CNN
-F 1 "10u" H 5850 2100 50  0000 L CNN
+F 1 "10uF" H 5850 2100 50  0000 L CNN
 F 2 "Capacitor_SMD:C_0402_1005Metric_Pad0.74x0.62mm_HandSolder" H 5800 2150 50  0001 C CNN
 F 3 "~" H 5800 2150 50  0001 C CNN
 F 4 "C15525" H 5800 2150 50  0001 C CNN "LCSC Part #"
+F 5 "581-0402ZD106MAT2A" H 5800 2150 50  0001 C CNN "Mouser"
 	1    5800 2150
 	1    0    0    -1
@@
 AR Path="/60860E11/60864A8F" Ref="C602"  Part="1"
 F 0 "C602" H 6150 2200 50  0000 L CNN
-F 1 "100n" H 6150 2100 50  0000 L CNN
+F 1 "0.1uF" H 6150 2100 50  0000 L CNN
 F 2 "Capacitor_SMD:C_0402_1005Metric_Pad0.74x0.62mm_HandSolder" H 6100 2150 50  0001 C CNN
 F 3 "~" H 6100 2150 50  0001 C CNN
 F 4 "C1525" H 6100 2150 50  0001 C CNN "LCSC Part #"
+F 5 "581-0402YD104K" H 6100 2150 50  0001 C CNN "Mouser"
 	1    6100 2150
 	1    0    0    -1
@@
 P 5150 3300
 F 0 "R602" H 5209 3346 50  0000 L CNN
-F 1 "1k" H 5209 3255 50  0000 L CNN
+F 1 "1kΩ" H 5209 3255 50  0000 L CNN
 F 2 "Resistor_SMD:R_0402_1005Metric_Pad0.72x0.64mm_HandSolder" H 5150 3300 50  0001 C CNN
 F 3 "~" H 5150 3300 50  0001 C CNN
@@
 P 4850 3300
 F 0 "R601" H 4909 3346 50  0000 L CNN
-F 1 "1k" H 4909 3255 50  0000 L CNN
+F 1 "1kΩ" H 4909 3255 50  0000 L CNN
 F 2 "Resistor_SMD:R_0402_1005Metric_Pad0.72x0.64mm_HandSolder" H 4850 3300 50  0001 C CNN
 F 3 "~" H 4850 3300 50  0001 C CNN
@@
 F 3 "~" V 7500 3850 50  0001 C CNN
 F 4 "C2286" H 7500 3850 50  0001 C CNN "LCSC Part #"
+F 5 "710-150060RS75020" H 7500 3850 50  0001 C CNN "Mouser"
 	1    7500 3850
 	0    -1   -1   0
@@
 AR Path="/60860E11/608D1F94" Ref="R603"  Part="1"
 F 0 "R603" H 7400 4050 50  0000 C CNN
-F 1 "1k5" H 7400 4150 50  0000 C CNN
+F 1 "1.5kΩ" H 7400 4150 50  0000 C CNN
 F 2 "Resistor_SMD:R_0603_1608Metric_Pad0.98x0.95mm_HandSolder" H 7500 4100 50  0001 C CNN
 F 3 "~" H 7500 4100 50  0001 C CNN

Commit message: Change part number
Parts:
- R601, R602: Mouser (none) -> 652-CR0402FX-1001GLF
- R603: Mouser (none) -> 755-KTR03EZPJ152
Changed lines of the file:
@@
 F 3 "~" H 5150 3300 50  0001 C CNN
 F 4 "C11702" H 5150 3300 50  0001 C CNN "LCSC Part #"
+F 5 "652-CR0402FX-1001GLF" H 5150 3300 50  0001 C CNN "Mouser"
 	1    5150 3300
 	1    0    0    -1
@@
 F 3 "~" H 4850 3300 50  0001 C CNN
 F 4 "C11702" H 4850 3300 50  0001 C CNN "LCSC Part #"
+F 5 "652-CR0402FX-1001GLF" H 4850 3300 50  0001 C CNN "Mouser"
 	1    4850 3300
 	1    0    0    -1
@@
 F 3 "~" H 7500 4100 50  0001 C CNN
 F 4 "C22843" H 7500 4100 50  0001 C CNN "LCSC Part #"
+F 5 "755-KTR03EZPJ152" H 7500 4100 50  0001 C CNN "Mouser"
 	1    7500 4100
 	-1   0    0    1
