File: Board_STM32F103C8T6/STM32F103C8T6/GPS.sch (KiCad schematic (older format))
At the start: 11 parts, among them J801 Conn_Coaxial, U801 MAX-M8Q

Commit message: Updated board design
work in progress
Parts:
- J801: footprint Board_02-Footprints:BWIPX-1-001E -> MyFootprints:BWIPX-1-001E
- L801: footprint Inductor_SMD:L_0402_1005Metric -> Inductor_SMD:L_0402_1005Metric_Pad0.77x0.64mm_HandSolder
Changed lines of the file:
@@
 F 0 "L801" V 7485 2650 50  0000 C CNN
 F 1 "100n" V 7394 2650 50  0000 C CNN
-F 2 "Inductor_SMD:L_0402_1005Metric" H 7300 2650 50  0001 C CNN
+F 2 "Inductor_SMD:L_0402_1005Metric_Pad0.77x0.64mm_HandSolder" H 7300 2650 50  0001 C CNN
 F 3 "~" H 7300 2650 50  0001 C CNN
 F 4 "C22726" H 7300 2650 50  0001 C CNN "LCSC Part #"
@@
 F 0 "J801" H 7950 3525 50  0000 L CNN
 F 1 "Conn_Coaxial" H 7950 3434 50  0000 L CNN
-F 2 "Board_02-Footprints:BWIPX-1-001E" H 7850 3550 50  0001 C CNN
+F 2 "MyFootprints:BWIPX-1-001E" H 7850 3550 50  0001 C CNN
 F 3 " ~" H 7850 3550 50  0001 C CNN
 F 4 "C496552" H 7850 3550 50  0001 C CNN "LCSC Part #"

Commit message: Changed Crystals
Parts:
- C801: value 10u -> 10uF; Mouser (none) -> 581-0402ZD106MAT2A
- C802, C803, C804: value 100n -> 0.1uF; Mouser (none) -> 581-0402YD104K
- C805: value 10n -> 0.01uF; Mouser (none) -> 581-0402ZC103KAT2A
- L801: value 100n -> 100nH; Mouser (none) -> 710-7447840210G
- R801, R802: value 0 -> 0kΩ
- R803: value 10 -> 10kΩ
Changed lines of the file:
@@
 P 4800 3000
 F 0 "R802" H 4859 3046 50  0000 L CNN
-F 1 "0" H 4859 2955 50  0000 L CNN
+F 1 "0kΩ" H 4859 2955 50  0000 L CNN
 F 2 "Resistor_SMD:R_0402_1005Metric_Pad0.72x0.64mm_HandSolder" H 4800 3000 50  0001 C CNN
 F 3 "~" H 4800 3000 50  0001 C CNN
@@
 P 4600 3000
 F 0 "R801" H 4659 3046 50  0000 L CNN
-F 1 "0" H 4659 2955 50  0000 L CNN
+F 1 "0kΩ" H 4659 2955 50  0000 L CNN
 F 2 "Resistor_SMD:R_0402_1005Metric_Pad0.72x0.64mm_HandSolder" H 4600 3000 50  0001 C CNN
 F 3 "~" H 4600 3000 50  0001 C CNN
@@
 P 6750 2650
 F 0 "R803" V 6650 2650 50  0000 C CNN
-F 1 "10" V 6850 2650 50  0000 C CNN
+F 1 "10kΩ" V 6850 2650 50  0000 C CNN
 F 2 "Resistor_SMD:R_0402_1005Metric_Pad0.72x0.64mm_HandSolder" H 6750 2650 50  0001 C CNN
 F 3 "~" H 6750 2650 50  0001 C CNN
@@
 P 7300 2650
 F 0 "L801" V 7485 2650 50  0000 C CNN
-F 1 "100n" V 7394 2650 50  0000 C CNN
+F 1 "100nH" V 7394 2650 50  0000 C CNN
 F 2 "Inductor_SMD:L_0402_1005Metric_Pad0.77x0.64mm_HandSolder" H 7300 2650 50  0001 C CNN
 F 3 "~" H 7300 2650 50  0001 C CNN
 F 4 "C22726" H 7300 2650 50  0001 C CNN "LCSC Part #"
+F 5 "710-7447840210G" H 7300 2650 50  0001 C CNN "Mouser"
 	1    7300 2650
 	0    -1   -1   0
@@
 P 7000 2800
 F 0 "C805" H 7092 2846 50  0000 L CNN
-F 1 "10n" H 7092 2755 50  0000 L CNN
+F 1 "0.01uF" H 7092 2755 50  0000 L CNN
 F 2 "Capacitor_SMD:C_0402_1005Metric_Pad0.74x0.62mm_HandSolder" H 7000 2800 50  0001 C CNN
 F 3 "~" H 7000 2800 50  0001 C CNN
 F 4 "C15195" H 7000 2800 50  0001 C CNN "LCSC Part #"
+F 5 "581-0402ZC103KAT2A" H 7000 2800 50  0001 C CNN "Mouser"
 	1    7000 2800
 	1    0    0    -1
@@
 P 5150 1750
 F 0 "C801" H 5200 1800 50  0000 L CNN
-F 1 "10u" H 5200 1700 50  0000 L CNN
+F 1 "10uF" H 5200 1700 50  0000 L CNN
 F 2 "Capacitor_SMD:C_0402_1005Metric_Pad0.74x0.62mm_HandSolder" H 5150 1750 50  0001 C CNN
 F 3 "~" H 5150 1750 50  0001 C CNN
 F 4 "C15525" H 5150 1750 50  0001 C CNN "LCSC Part #"
+F 5 "581-0402ZD106MAT2A" H 5150 1750 50  0001 C CNN "Mouser"
 	1    5150 1750
 	1    0    0    -1
@@
 P 5450 1750
 F 0 "C802" H 5500 1800 50  0000 L CNN
-F 1 "100n" H 5500 1700 50  0000 L CNN
+F 1 "0.1uF" H 5500 1700 50  0000 L CNN
 F 2 "Capacitor_SMD:C_0402_1005Metric_Pad0.74x0.62mm_HandSolder" H 5450 1750 50  0001 C CNN
 F 3 "~" H 5450 1750 50  0001 C CNN
 F 4 "C1525" H 5450 1750 50  0001 C CNN "LCSC Part #"
+F 5 "581-0402YD104K" H 5450 1750 50  0001 C CNN "Mouser"
 	1    5450 1750
 	1    0    0    -1
@@
 P 5800 1750
 F 0 "C803" H 5850 1800 50  0000 L CNN
-F 1 "100n" H 5850 1700 50  0000 L CNN
+F 1 "0.1uF" H 5850 1700 50  0000 L CNN
 F 2 "Capacitor_SMD:C_0402_1005Metric_Pad0.74x0.62mm_HandSolder" H 5800 1750 50  0001 C CNN
 F 3 "~" H 5800 1750 50  0001 C CNN
 F 4 "C1525" H 5800 1750 50  0001 C CNN "LCSC Part #"
+F 5 "581-0402YD104K" H 5800 1750 50  0001 C CNN "Mouser"
 	1    5800 1750
 	1    0    0    -1
@@
 P 6150 1750
 F 0 "C804" H 6200 1800 50  0000 L CNN
-F 1 "100n" H 6200 1700 50  0000 L CNN
+F 1 "0.1uF" H 6200 1700 50  0000 L CNN
 F 2 "Capacitor_SMD:C_0402_1005Metric_Pad0.74x0.62mm_HandSolder" H 6150 1750 50  0001 C CNN
 F 3 "~" H 6150 1750 50  0001 C CNN
 F 4 "C1525" H 6150 1750 50  0001 C CNN "LCSC Part #"
+F 5 "581-0402YD104K" H 6150 1750 50  0001 C CNN "Mouser"
 	1    6150 1750
 	1    0    0    -1

Commit message: Change part number
Parts:
- J801: footprint MyFootprints:BWIPX-1-001E -> Connector_Coaxial:SMA_Molex_73251-2200_Horizontal; LCSC Part # C496552 -> (none); Mouser (none) -> 538-73391-0080
- R801, R802: Mouser (none) -> 652-CR0402-J/-000GLF
- R803: LCSC Part # C25077 -> (none); Mouser (none) -> 71-CRCW040210K0FKEDC
Changed lines of the file:
@@
 F 3 "~" H 4800 3000 50  0001 C CNN
 F 4 "C17168" H 4800 3000 50  0001 C CNN "LCSC Part #"
+F 5 "652-CR0402-J/-000GLF" H 4800 3000 50  0001 C CNN "Mouser"
 	1    4800 3000
 	1    0    0    -1
@@
 F 3 "~" H 4600 3000 50  0001 C CNN
 F 4 "C17168" H 4600 3000 50  0001 C CNN "LCSC Part #"
+F 5 "652-CR0402-J/-000GLF" H 4600 3000 50  0001 C CNN "Mouser"
 	1    4600 3000
 	1    0    0    -1
@@
 F 2 "Resistor_SMD:R_0402_1005Metric_Pad0.72x0.64mm_HandSolder" H 6750 2650 50  0001 C CNN
 F 3 "~" H 6750 2650 50  0001 C CNN
-F 4 "C25077" H 6750 2650 50  0001 C CNN "LCSC Part #"
+F 4 "" H 6750 2650 50  0001 C CNN "LCSC Part #"
+F 5 "71-CRCW040210K0FKEDC" H 6750 2650 50  0001 C CNN "Mouser"
 	1    6750 2650
 	0    1    1    0
@@
 F 0 "J801" H 7950 3525 50  0000 L CNN
 F 1 "Conn_Coaxial" H 7950 3434 50  0000 L CNN
-F 2 "MyFootprints:BWIPX-1-001E" H 7850 3550 50  0001 C CNN
+F 2 "Connector_Coaxial:SMA_Molex_73251-2200_Horizontal" H 7850 3550 50  0001 C CNN
 F 3 " ~" H 7850 3550 50  0001 C CNN
-F 4 "C496552" H 7850 3550 50  0001 C CNN "LCSC Part #"
+F 4 "" H 7850 3550 50  0001 C CNN "LCSC Part #"
+F 5 "538-73391-0080" H 7850 3550 50  0001 C CNN "Mouser"
 	1    7850 3550
 	1    0    0    -1
