File: Board_STM32F103C8T6/STM32F103C8T6/Power.sch (KiCad schematic (older format))
At the start: 9 parts, among them Q201 AO3401A, U201 LD1117S33TR_SOT223

Commit message: Updated board design
work in progress
Parts:
- FB201: footprint Inductor_SMD:L_0805_2012Metric -> Inductor_SMD:L_1206_3216Metric_Pad1.22x1.90mm_HandSolder
Changed lines of the file:
@@
 F 0 "FB201" V 3900 2100 50  0000 C CNN
 F 1 "600 @ 600 MHz" V 4150 2100 50  0000 C CNN
-F 2 "Inductor_SMD:L_0805_2012Metric" V 3980 2100 50  0001 C CNN
+F 2 "Inductor_SMD:L_1206_3216Metric_Pad1.22x1.90mm_HandSolder" V 3980 2100 50  0001 C CNN
 F 3 "~" H 4050 2100 50  0001 C CNN
 F 4 "C1017" H 4050 2100 50  0001 C CNN "LCSC Part #"

Commit message: added files to product pcb
Parts:
- U201: value LD1117S33TR_SOT223 -> LD1117S33TR; LCSC Part # (none) -> C86781
Changed lines of the file:
@@
 P 5300 2100
 F 0 "U201" H 5300 2342 50  0000 C CNN
-F 1 "LD1117S33TR_SOT223" H 5300 2251 50  0000 C CNN
+F 1 "LD1117S33TR" H 5300 2251 50  0000 C CNN
 F 2 "Package_TO_SOT_SMD:SOT-223-3_TabPin2" H 5300 2300 50  0001 C CNN
 F 3 "http://www.st.com/st-web-ui/static/active/en/resource/technical/document/datasheet/CD00000544.pdf" H 5400 1850 50  0001 C CNN
+F 4 "C86781" H 5300 2100 50  0001 C CNN "LCSC Part #"
 	1    5300 2100
 	1    0    0    -1

Commit message: Changed Crystals
Parts:
- C201: value 100n -> 0.1uF; Mouser (none) -> 581-1206VC104KAT2A
- C202: value 10u -> 10uF; Mouser (none) -> 581-1206DD106KAT2A
- D201: Mouser (none) -> 833-B5819W-TP
- D202: Mouser (none) -> 710-150060GS75020
- F201: Mouser (none) -> 576-1206L050YR
- FB201: Mouser (none) -> 70-ILHB1206ER601V
- R201: value 1k5 -> 1.5kΩ
- U201: Mouser (none) -> 511-LD1117S33
Changed lines of the file:
@@
 F 3 "~" H 2600 2100 50  0001 C CNN
 F 4 "C70068" H 2600 2100 50  0001 C CNN "LCSC Part #"
+F 5 "576-1206L050YR" H 2600 2100 50  0001 C CNN "Mouser"
 	1    2600 2100
 	0    1    1    0
@@
 F 3 "~" H 4050 2100 50  0001 C CNN
 F 4 "C1017" H 4050 2100 50  0001 C CNN "LCSC Part #"
+F 5 "70-ILHB1206ER601V" H 4050 2100 50  0001 C CNN "Mouser"
 	1    4050 2100
 	0    1    1    0
@@
 P 4450 2250
 F 0 "C201" H 4500 2300 50  0000 L CNN
-F 1 "100n" H 4500 2200 50  0000 L CNN
+F 1 "0.1uF" H 4500 2200 50  0000 L CNN
 F 2 "Capacitor_SMD:C_1206_3216Metric_Pad1.33x1.80mm_HandSolder" H 4450 2250 50  0001 C CNN
 F 3 "~" H 4450 2250 50  0001 C CNN
 F 4 "C13585" H 4450 2250 50  0001 C CNN "LCSC Part #"
+F 5 "581-1206VC104KAT2A" H 4450 2250 50  0001 C CNN "Mouser"
 	1    4450 2250
 	1    0    0    -1
@@
 F 3 "https://datasheet.lcsc.com/szlcsc/Changjiang-Electronics-Tech-CJ-B5819W_C8598.pdf" V 3500 1950 50  0001 C CNN
 F 4 "C8598" H 3500 1950 50  0001 C CNN "LCSC Part #"
+F 5 "833-B5819W-TP" H 3500 1950 50  0001 C CNN "Mouser"
 	1    3500 1950
 	0    -1   -1   0
@@
 P 7050 2450
 F 0 "R201" H 7109 2496 50  0000 L CNN
-F 1 "1k5" H 7109 2405 50  0000 L CNN
+F 1 "1.5kΩ" H 7109 2405 50  0000 L CNN
 F 2 "Resistor_SMD:R_0603_1608Metric_Pad0.98x0.95mm_HandSolder" H 7050 2450 50  0001 C CNN
 F 3 "~" H 7050 2450 50  0001 C CNN
@@
 F 3 "~" V 7050 2250 50  0001 C CNN
 F 4 "C72043" H 7050 2250 50  0001 C CNN "LCSC Part #"
+F 5 "710-150060GS75020" H 7050 2250 50  0001 C CNN "Mouser"
 	1    7050 2250
 	0    -1   -1   0
@@
 F 3 "http://www.st.com/st-web-ui/static/active/en/resource/technical/document/datasheet/CD00000544.pdf" H 5400 1850 50  0001 C CNN
 F 4 "C86781" H 5300 2100 50  0001 C CNN "LCSC Part #"
+F 5 "511-LD1117S33" H 5300 2100 50  0001 C CNN "Mouser"
 	1    5300 2100
 	1    0    0    -1
@@
 P 6150 2250
 F 0 "C202" H 6200 2300 50  0000 L CNN
-F 1 "10u" H 6200 2200 50  0000 L CNN
+F 1 "10uF" H 6200 2200 50  0000 L CNN
 F 2 "Capacitor_SMD:C_1206_3216Metric_Pad1.33x1.80mm_HandSolder" H 6150 2250 50  0001 C CNN
 F 3 "~" H 6150 2250 50  0001 C CNN
 F 4 "C13585" H 6150 2250 50  0001 C CNN "LCSC Part #"
+F 5 "581-1206DD106KAT2A" H 6150 2250 50  0001 C CNN "Mouser"
 	1    6150 2250
 	1    0    0    -1

Commit message: Change part number
Parts:
- Q201: value AO3401A -> SI2301CDS-T1-BE3; footprint Package_TO_SOT_SMD:SOT-23 -> Package_TO_SOT_SMD:SOT-23_Handsoldering; LCSC Part # C306862 -> (none); Mouser (none) -> 78-SI2301CDS-T1-BE3
- R201: Mouser (none) -> 755-KTR03EZPJ152
Other:
- note added: "AMS1117-33"
Changed lines of the file:
@@
 P 3050 2200
 F 0 "Q201" V 3392 2200 50  0000 C CNN
-F 1 "AO3401A" V 3301 2200 50  0000 C CNN
-F 2 "Package_TO_SOT_SMD:SOT-23" H 3250 2125 50  0001 L CIN
-F 3 "http://www.aosmd.com/pdfs/datasheet/AO3401A.pdf" H 3050 2200 50  0001 L CNN
-F 4 "C306862" H 3050 2200 50  0001 C CNN "LCSC Part #"
+F 1 "SI2301CDS-T1-BE3" V 3301 2200 50  0000 C CNN
+F 2 "Package_TO_SOT_SMD:SOT-23_Handsoldering" H 3250 2125 50  0001 L CIN
+F 3 "" H 3050 2200 50  0001 L CNN
+F 4 "" H 3050 2200 50  0001 C CNN "LCSC Part #"
+F 5 "78-SI2301CDS-T1-BE3" H 3050 2200 50  0001 C CNN "Mouser"
 	1    3050 2200
 	0    -1   -1   0
@@
 F 3 "~" H 7050 2450 50  0001 C CNN
 F 4 "C22843" H 7050 2450 50  0001 C CNN "LCSC Part #"
+F 5 "755-KTR03EZPJ152" H 7050 2450 50  0001 C CNN "Mouser"
 	1    7050 2450
 	1    0    0    -1
@@
 Text Notes 2200 1550 0    50   ~ 0
 VBAT = 3 x 1,5V\n(4.5V)
+Text Notes 5050 1700 0    50   ~ 0
+AMS1117-33
 $EndSCHEMATC
