File: Board_STM32F103C8T6/STM32F103C8T6/Connectors.sch (KiCad schematic (older format))
At the start: 12 parts, among them J401 BATTERY, J402 I2C, J403 H2O, J404 USB_B_Micro, J405 SWD, J406 USART1, J407 CIRCUIT_SENSOR, J408 BLUETOOTH, J409 RPM, J410 POWER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

Commit message: Improved PCB layout
Parts:
- added C402, C403: 47p, Capacitor_SMD:C_0402_1005Metric_Pad0.74x0.62mm_HandSolder, symbol Device:C_Small
- added R401, R402: 22, Resistor_SMD:R_0402_1005Metric_Pad0.72x0.64mm_HandSolder, symbol Device:R_Small
- C401: value 10u -> 100n
Connections:
- wire segments 22 -> 40
Changed lines of the file:
@@
-$EndComp
-$Comp
-L power:+5V #PWR0412
-U 1 1 6090DD66
-P 5450 2100
-F 0 "#PWR0412" H 5450 1950 50  0001 C CNN
-F 1 "+5V" H 5465 2273 50  0000 C CNN
-F 2 "" H 5450 2100 50  0001 C CNN
-F 3 "" H 5450 2100 50  0001 C CNN
-	1    5450 2100
-	1    0    0    -1
-$EndComp
-$Comp
-L power:GND #PWR0413
-U 1 1 608EE482
-P 5450 2300
-F 0 "#PWR0413" H 5450 2050 50  0001 C CNN
-F 1 "GND" H 5455 2127 50  0000 C CNN
-F 2 "" H 5450 2300 50  0001 C CNN
-F 3 "" H 5450 2300 50  0001 C CNN
-	1    5450 2300
-	1    0    0    -1
 $EndComp
 $Comp
 L Device:C_Small C401
 U 1 1 608EDDAA
-P 5450 2200
-F 0 "C401" H 5500 2250 50  0000 L CNN
-F 1 "10u" H 5500 2150 50  0000 L CNN
-F 2 "Capacitor_SMD:C_0402_1005Metric_Pad0.74x0.62mm_HandSolder" H 5450 2200 50  0001 C CNN
-F 3 "~" H 5450 2200 50  0001 C CNN
-F 4 "C15525" H 5450 2200 50  0001 C CNN "LCSC Part #"
-	1    5450 2200
-	1    0    0    -1
-$EndComp
-$Comp
-L power:+5V #PWR0410
-U 1 1 608732C4
-P 5150 2600
-F 0 "#PWR0410" H 5150 2450 50  0001 C CNN
-F 1 "+5V" H 5165 2773 50  0000 C CNN
-F 2 "" H 5150 2600 50  0001 C CNN
-F 3 "" H 5150 2600 50  0001 C CNN
-	1    5150 2600
+P 7300 3050
+F 0 "C401" H 7350 3100 50  0000 L CNN
+F 1 "100n" H 7350 3000 50  0000 L CNN
+F 2 "Capacitor_SMD:C_0402_1005Metric_Pad0.74x0.62mm_HandSolder" H 7300 3050 50  0001 C CNN
+F 3 "~" H 7300 3050 50  0001 C CNN
+F 4 "C15525" H 7300 3050 50  0001 C CNN "LCSC Part #"
+	1    7300 3050
 	1    0    0    -1
 $EndComp
@@
 L power:GND #PWR0411
 U 1 1 60872E86
-P 5150 3400
-F 0 "#PWR0411" H 5150 3150 50  0001 C CNN
-F 1 "GND" H 5155 3227 50  0000 C CNN
-F 2 "" H 5150 3400 50  0001 C CNN
-F 3 "" H 5150 3400 50  0001 C CNN
-	1    5150 3400
-	1    0    0    -1
-$EndComp
-Text GLabel 5550 3100 2    50   Input ~ 0
+P 5700 3500
+F 0 "#PWR0411" H 5700 3250 50  0001 C CNN
+F 1 "GND" H 5705 3327 50  0000 C CNN
+F 2 "" H 5700 3500 50  0001 C CNN
+F 3 "" H 5700 3500 50  0001 C CNN
+	1    5700 3500
+	1    0    0    -1
+$EndComp
+Text GLabel 6100 3050 2    50   Input ~ 0
 USB_CONN_D+
-Text GLabel 4750 3100 0    50   Input ~ 0
+Text GLabel 5300 3050 0    50   Input ~ 0
 USB_CONN_D-
-$Comp
-L Power_Protection:USBLC6-2SC6 U401
-U 1 1 6086FC62
-P 5150 3000
-F 0 "U401" H 5400 3350 50  0000 C CNN
-F 1 "USBLC6-2SC6" H 5450 2650 50  0000 C CNN
-F 2 "Package_TO_SOT_SMD:SOT-23-6" H 5150 2500 50  0001 C CNN
-F 3 "https://www.st.com/resource/en/datasheet/usblc6-2.pdf" H 5350 3350 50  0001 C CNN
-F 4 "C558442" H 5150 3000 50  0001 C CNN "LCSC Part #"
-	1    5150 3000
-	1    0    0    -1
-$EndComp
-Text GLabel 4750 2900 0    50   Input ~ 0
+Text GLabel 4450 2850 0    50   Input ~ 0
 USB_D-
-Text GLabel 5550 2900 2    50   Input ~ 0
+Text GLabel 6850 2850 2    50   Input ~ 0
 USB_D+
 Wire Wire Line
@@
 	1    0    0    -1
 $EndComp
+$Comp
+L power:+3.3V #PWR0102
+U 1 1 61D1BB27
+P 5700 2400
+F 0 "#PWR0102" H 5700 2250 50  0001 C CNN
+F 1 "+3.3V" H 5715 2573 50  0000 C CNN
+F 2 "" H 5700 2400 50  0001 C CNN
+F 3 "" H 5700 2400 50  0001 C CNN
+	1    5700 2400
+	1    0    0    -1
+$EndComp
+$Comp
+L Power_Protection:USBLC6-2SC6 U401
+U 1 1 6086FC62
+P 5700 2950
+F 0 "U401" H 5950 3300 50  0000 C CNN
+F 1 "USBLC6-2SC6" H 6000 2600 50  0000 C CNN
+F 2 "Package_TO_SOT_SMD:SOT-23-6" H 5700 2450 50  0001 C CNN
+F 3 "https://www.st.com/resource/en/datasheet/usblc6-2.pdf" H 5900 3300 50  0001 C CNN
+F 4 "C558442" H 5700 2950 50  0001 C CNN "LCSC Part #"
+	1    5700 2950
+	1    0    0    -1
+$EndComp
+$Comp
+L Device:R_Small R402
+U 1 1 61D28325
+P 6200 2850
+F 0 "R402" V 6004 2850 50  0000 C CNN
+F 1 "22" V 6095 2850 50  0000 C CNN
+F 2 "Resistor_SMD:R_0402_1005Metric_Pad0.72x0.64mm_HandSolder" H 6200 2850 50  0001 C CNN
+F 3 "~" H 6200 2850 50  0001 C CNN
+	1    6200 2850
+	0    1    1    0
+$EndComp
+$Comp
+L Device:R_Small R401
+U 1 1 61D2919D
+P 5200 2850
+F 0 "R401" V 5004 2850 50  0000 C CNN
+F 1 "22" V 5095 2850 50  0000 C CNN
+F 2 "Resistor_SMD:R_0402_1005Metric_Pad0.72x0.64mm_HandSolder" H 5200 2850 50  0001 C CNN
+F 3 "~" H 5200 2850 50  0001 C CNN
+	1    5200 2850
+	0    1    1    0
+$EndComp
+$Comp
+L Device:C_Small C403
+U 1 1 61D2E57B
+P 6800 3050
+F 0 "C403" H 6850 3100 50  0000 L CNN
+F 1 "47p" H 6850 3000 50  0000 L CNN
+F 2 "Capacitor_SMD:C_0402_1005Metric_Pad0.74x0.62mm_HandSolder" H 6800 3050 50  0001 C CNN
+F 3 "~" H 6800 3050 50  0001 C CNN
+F 4 "C15525" H 6800 3050 50  0001 C CNN "LCSC Part #"
+	1    6800 3050
+	1    0    0    -1
+$EndComp
+Wire Wire Line
+	6300 2850 6800 2850
+Wire Wire Line
+	6800 2950 6800 2850
+Wire Wire Line
+	7300 2450 7300 2950
+$Comp
+L Device:C_Small C402
+U 1 1 61D3175C
+P 4500 3050
+F 0 "C402" H 4550 3100 50  0000 L CNN
+F 1 "47p" H 4550 3000 50  0000 L CNN
+F 2 "Capacitor_SMD:C_0402_1005Metric_Pad0.74x0.62mm_HandSolder" H 4500 3050 50  0001 C CNN
+F 3 "~" H 4500 3050 50  0001 C CNN
+F 4 "C15525" H 4500 3050 50  0001 C CNN "LCSC Part #"
+	1    4500 3050
+	1    0    0    -1
+$EndComp
+Wire Wire Line
+	4500 2950 4500 2850
+Wire Wire Line
+	4500 2850 5100 2850
+Wire Wire Line
+	4500 3150 4500 3400
+Wire Wire Line
+	4500 3400 5700 3400
+Wire Wire Line
+	5700 3400 5700 3500
+Wire Wire Line
+	5700 3400 5700 3350
+Connection ~ 5700 3400
+Wire Wire Line
+	5700 3400 6800 3400
+Wire Wire Line
+	6800 3400 6800 3150
+Wire Wire Line
+	7300 3400 7300 3150
+Wire Wire Line
+	4450 2850 4500 2850
+Connection ~ 4500 2850
+Wire Wire Line
+	5700 2400 5700 2450
+Wire Wire Line
+	5700 2450 7300 2450
+Connection ~ 5700 2450
+Wire Wire Line
+	5700 2450 5700 2550
+Wire Wire Line
+	7300 3400 6800 3400
+Connection ~ 6800 3400
+Wire Wire Line
+	6850 2850 6800 2850
+Connection ~ 6800 2850
 $EndSCHEMATC

Commit message: added files to product pcb
Parts:
- C401: LCSC Part # C15525 -> C1525
- C402, C403: LCSC Part # C15525 -> C1567
- R401, R402: LCSC Part # (none) -> C25092
Changed lines of the file:
@@
 F 2 "Capacitor_SMD:C_0402_1005Metric_Pad0.74x0.62mm_HandSolder" H 7300 3050 50  0001 C CNN
 F 3 "~" H 7300 3050 50  0001 C CNN
-F 4 "C15525" H 7300 3050 50  0001 C CNN "LCSC Part #"
+F 4 "C1525" H 7300 3050 50  0001 C CNN "LCSC Part #"
 	1    7300 3050
 	1    0    0    -1
@@
 F 2 "Resistor_SMD:R_0402_1005Metric_Pad0.72x0.64mm_HandSolder" H 6200 2850 50  0001 C CNN
 F 3 "~" H 6200 2850 50  0001 C CNN
+F 4 "C25092" H 6200 2850 50  0001 C CNN "LCSC Part #"
 	1    6200 2850
 	0    1    1    0
@@
 F 2 "Resistor_SMD:R_0402_1005Metric_Pad0.72x0.64mm_HandSolder" H 5200 2850 50  0001 C CNN
 F 3 "~" H 5200 2850 50  0001 C CNN
+F 4 "C25092" H 5200 2850 50  0001 C CNN "LCSC Part #"
 	1    5200 2850
 	0    1    1    0
@@
 F 2 "Capacitor_SMD:C_0402_1005Metric_Pad0.74x0.62mm_HandSolder" H 6800 3050 50  0001 C CNN
 F 3 "~" H 6800 3050 50  0001 C CNN
-F 4 "C15525" H 6800 3050 50  0001 C CNN "LCSC Part #"
+F 4 "C1567" H 6800 3050 50  0001 C CNN "LCSC Part #"
 	1    6800 3050
 	1    0    0    -1
@@
 F 2 "Capacitor_SMD:C_0402_1005Metric_Pad0.74x0.62mm_HandSolder" H 4500 3050 50  0001 C CNN
 F 3 "~" H 4500 3050 50  0001 C CNN
-F 4 "C15525" H 4500 3050 50  0001 C CNN "LCSC Part #"
+F 4 "C1567" H 4500 3050 50  0001 C CNN "LCSC Part #"
 	1    4500 3050
 	1    0    0    -1

Commit message: Changed Crystals
Parts:
- C401: value 100n -> 0.1uF; Mouser (none) -> 581-0402YD104K
- C402, C403: value 47p -> 47pF; Mouser (none) -> 581-0402ZA470JAT2A
- J404: Mouser (none) -> 710-614105150721
- R401, R402: value 22 -> 22kΩ
- U401: Mouser (none) -> 511-USBLC6-2SC6
Changed lines of the file:
@@
 P 7300 3050
 F 0 "C401" H 7350 3100 50  0000 L CNN
-F 1 "100n" H 7350 3000 50  0000 L CNN
+F 1 "0.1uF" H 7350 3000 50  0000 L CNN
 F 2 "Capacitor_SMD:C_0402_1005Metric_Pad0.74x0.62mm_HandSolder" H 7300 3050 50  0001 C CNN
 F 3 "~" H 7300 3050 50  0001 C CNN
 F 4 "C1525" H 7300 3050 50  0001 C CNN "LCSC Part #"
+F 5 "581-0402YD104K" H 7300 3050 50  0001 C CNN "Mouser"
 	1    7300 3050
 	1    0    0    -1
@@
 F 3 "~" H 2850 2800 50  0001 C CNN
 F 4 "C40943" H 2700 2850 50  0001 C CNN "LCSC Part #"
+F 5 "710-614105150721" H 2700 2850 50  0001 C CNN "Mouser"
 	1    2700 2850
 	1    0    0    -1
@@
 F 3 "https://www.st.com/resource/en/datasheet/usblc6-2.pdf" H 5900 3300 50  0001 C CNN
 F 4 "C558442" H 5700 2950 50  0001 C CNN "LCSC Part #"
+F 5 "511-USBLC6-2SC6" H 5700 2950 50  0001 C CNN "Mouser"
 	1    5700 2950
 	1    0    0    -1
@@
 P 6200 2850
 F 0 "R402" V 6004 2850 50  0000 C CNN
-F 1 "22" V 6095 2850 50  0000 C CNN
+F 1 "22kΩ" V 6095 2850 50  0000 C CNN
 F 2 "Resistor_SMD:R_0402_1005Metric_Pad0.72x0.64mm_HandSolder" H 6200 2850 50  0001 C CNN
 F 3 "~" H 6200 2850 50  0001 C CNN
@@
 P 5200 2850
 F 0 "R401" V 5004 2850 50  0000 C CNN
-F 1 "22" V 5095 2850 50  0000 C CNN
+F 1 "22kΩ" V 5095 2850 50  0000 C CNN
 F 2 "Resistor_SMD:R_0402_1005Metric_Pad0.72x0.64mm_HandSolder" H 5200 2850 50  0001 C CNN
 F 3 "~" H 5200 2850 50  0001 C CNN
@@
 P 6800 3050
 F 0 "C403" H 6850 3100 50  0000 L CNN
-F 1 "47p" H 6850 3000 50  0000 L CNN
+F 1 "47pF" H 6850 3000 50  0000 L CNN
 F 2 "Capacitor_SMD:C_0402_1005Metric_Pad0.74x0.62mm_HandSolder" H 6800 3050 50  0001 C CNN
 F 3 "~" H 6800 3050 50  0001 C CNN
 F 4 "C1567" H 6800 3050 50  0001 C CNN "LCSC Part #"
+F 5 "581-0402ZA470JAT2A" H 6800 3050 50  0001 C CNN "Mouser"
 	1    6800 3050
 	1    0    0    -1
@@
 P 4500 3050
 F 0 "C402" H 4550 3100 50  0000 L CNN
-F 1 "47p" H 4550 3000 50  0000 L CNN
+F 1 "47pF" H 4550 3000 50  0000 L CNN
 F 2 "Capacitor_SMD:C_0402_1005Metric_Pad0.74x0.62mm_HandSolder" H 4500 3050 50  0001 C CNN
 F 3 "~" H 4500 3050 50  0001 C CNN
 F 4 "C1567" H 4500 3050 50  0001 C CNN "LCSC Part #"
+F 5 "581-0402ZA470JAT2A" H 4500 3050 50  0001 C CNN "Mouser"
 	1    4500 3050
 	1    0    0    -1

Commit message: Change part number
Parts:
- R401, R402: Mouser (none) -> 652-CR0402FX-2202GLF
Changed lines of the file:
@@
 F 3 "~" H 6200 2850 50  0001 C CNN
 F 4 "C25092" H 6200 2850 50  0001 C CNN "LCSC Part #"
+F 5 "652-CR0402FX-2202GLF" H 6200 2850 50  0001 C CNN "Mouser"
 	1    6200 2850
 	0    1    1    0
@@
 F 3 "~" H 5200 2850 50  0001 C CNN
 F 4 "C25092" H 5200 2850 50  0001 C CNN "LCSC Part #"
+F 5 "652-CR0402FX-2202GLF" H 5200 2850 50  0001 C CNN "Mouser"
 	1    5200 2850
 	0    1    1    0

Commit message: Added descriptions
Parts:
- removed J404: USB_B_Micro, Connector_USB:USB_Micro-B_Wuerth_629105150521, symbol Connector:USB_B_Micro
- added J404: USB_C_Receptacle_USB2.0, Connector_USB:USB_C_Receptacle_Palconn_UTC16-G, symbol Connector:USB_C_Receptacle_USB2.0
- added R403, R404: 5.1kΩ, Resistor_SMD:R_0402_1005Metric_Pad0.72x0.64mm_HandSolder, symbol Device:R_Small
Connections:
- wire segments 40 -> 60
- no-connect marks 4 -> 5
