File: Board_STM32F103C8T6/STM32F103C8T6/MCU.sch (KiCad schematic (older format))
At the start: 50 parts, among them J301 BOOT, Q301 VP0610T, U301 W25Q128JVS, U302 STM32F103C8T6, Y301 8Mhz, Y302 32.768KHZ

Commit message: Updated board design
work in progress
Parts:
- H307, H308, H309: footprint Board_02-Footprints:JLCPCB-Tooling-Hole -> MyFootprints:JLCPCB-Tooling-Hole
- L301: footprint Inductor_SMD:L_0402_1005Metric -> Inductor_SMD:L_0402_1005Metric_Pad0.77x0.64mm_HandSolder
- Q301: value VP0610T -> AO3401A; symbol Transistor_FET:VP0610T -> Transistor_FET:AO3401A
- Y301: footprint Crystal:Crystal_SMD_5032-2Pin_5.0x3.2mm -> Crystal:Crystal_SMD_5032-2Pin_5.0x3.2mm_HandSoldering
Changed lines of the file:
@@
 F 0 "L301" V 2700 1100 50  0000 C CNN
 F 1 "39n" V 2600 1100 50  0000 C CNN
-F 2 "Inductor_SMD:L_0402_1005Metric" H 2650 1100 50  0001 C CNN
+F 2 "Inductor_SMD:L_0402_1005Metric_Pad0.77x0.64mm_HandSolder" H 2650 1100 50  0001 C CNN
 F 3 "~" H 2650 1100 50  0001 C CNN
 F 4 "C26443" H 2650 1100 50  0001 C CNN "LCSC Part #"
@@
 F 0 "Y301" H 4850 5025 50  0000 C CNN
 F 1 "8Mhz" H 4850 4934 50  0000 C CNN
-F 2 "Crystal:Crystal_SMD_5032-2Pin_5.0x3.2mm" H 4850 4800 50  0001 C CNN
+F 2 "Crystal:Crystal_SMD_5032-2Pin_5.0x3.2mm_HandSoldering" H 4850 4800 50  0001 C CNN
 F 3 "https://datasheet.lcsc.com/szlcsc/1903061615_Yangxing-Tech-X50328MSB2GI_C115962.pdf" H 4850 4800 50  0001 C CNN
 F 4 "" H 4850 4800 50  0001 C CNN "NAME"
@@
 F 0 "H307" H 10300 5846 50  0000 L CNN
 F 1 "MountingHole" H 10300 5755 50  0000 L CNN
-F 2 "Board_02-Footprints:JLCPCB-Tooling-Hole" H 10200 5800 50  0001 C CNN
+F 2 "MyFootprints:JLCPCB-Tooling-Hole" H 10200 5800 50  0001 C CNN
 F 3 "~" H 10200 5800 50  0001 C CNN
 	1    10200 5800
@@
 F 0 "H308" H 10300 6046 50  0000 L CNN
 F 1 "MountingHole" H 10300 5955 50  0000 L CNN
-F 2 "Board_02-Footprints:JLCPCB-Tooling-Hole" H 10200 6000 50  0001 C CNN
+F 2 "MyFootprints:JLCPCB-Tooling-Hole" H 10200 6000 50  0001 C CNN
 F 3 "~" H 10200 6000 50  0001 C CNN
 	1    10200 6000
@@
 F 0 "H309" H 10300 6246 50  0000 L CNN
 F 1 "MountingHole" H 10300 6155 50  0000 L CNN
-F 2 "Board_02-Footprints:JLCPCB-Tooling-Hole" H 10200 6200 50  0001 C CNN
+F 2 "MyFootprints:JLCPCB-Tooling-Hole" H 10200 6200 50  0001 C CNN
 F 3 "~" H 10200 6200 50  0001 C CNN
 	1    10200 6200
@@
 	10050 2000 10050 2100
 $Comp
-L Transistor_FET:VP0610T Q301
+L Transistor_FET:AO3401A Q301
 U 1 1 61D4997A
 P 10150 2300
 F 0 "Q301" H 10355 2254 50  0000 L CNN
-F 1 "VP0610T" H 10355 2345 50  0000 L CNN
+F 1 "AO3401A" H 10355 2345 50  0000 L CNN
 F 2 "Package_TO_SOT_SMD:SOT-23" H 10350 2225 50  0001 L CIN
-F 3 "http://www.vishay.com/docs/70209/70209.pdf" H 10150 2300 50  0001 L CNN
+F 3 "http://www.aosmd.com/pdfs/datasheet/AO3401A.pdf" H 10150 2300 50  0001 L CNN
 	1    10150 2300
 	-1   0    0    1

Commit message: Improved PCB layout
Parts:
- removed Q301: AO3401A, Package_TO_SOT_SMD:SOT-23, symbol Transistor_FET:AO3401A
- added Q301: BSS123, Package_TO_SOT_SMD:SOT-23, symbol Transistor_FET:BSS123
Connections:
- wire segments 135 -> 139
Changed lines of the file:
@@
 Text GLabel 2700 6400 2    50   Input ~ 0
 H2O_NTC+
-Text GLabel 10050 2800 3    50   Input ~ 0
+Text GLabel 10650 2050 2    50   Input ~ 0
 USB_D+
 $Comp
 L Device:R_Small R319
 U 1 1 608E4215
-P 10050 2650
+P 10600 1800
 AR Path="/607F2E3B/608E4215" Ref="R319"  Part="1"
 AR Path="/608AF770/608E4215" Ref="R?"  Part="1"
-F 0 "R319" H 9950 2600 50  0000 C CNN
-F 1 "1k5" H 9900 2700 50  0000 C CNN
-F 2 "Resistor_SMD:R_0402_1005Metric_Pad0.72x0.64mm_HandSolder" H 10050 2650 50  0001 C CNN
-F 3 "~" H 10050 2650 50  0001 C CNN
-F 4 "C25867" H 10050 2650 50  0001 C CNN "LCSC Part #"
-	1    10050 2650
+F 0 "R319" H 10500 1750 50  0000 C CNN
+F 1 "1k5" H 10450 1850 50  0000 C CNN
+F 2 "Resistor_SMD:R_0402_1005Metric_Pad0.72x0.64mm_HandSolder" H 10600 1800 50  0001 C CNN
+F 3 "~" H 10600 1800 50  0001 C CNN
+F 4 "C25867" H 10600 1800 50  0001 C CNN "LCSC Part #"
+	1    10600 1800
 	-1   0    0    1
 $EndComp
 Wire Wire Line
-	10050 2550 10050 2500
-Wire Wire Line
-	10050 2800 10050 2750
+	10600 1700 10600 1650
 Text GLabel 1400 5800 0    50   Input ~ 0
 GPS_PPS
@@
 Text GLabel 2700 7200 2    50   Input ~ 0
 USB_EN
-Text GLabel 10750 2300 2    50   Input ~ 0
+Text GLabel 10000 2350 0    50   Input ~ 0
 USB_EN
 Wire Bus Line
@@
 L power:+3.3V #PWR0322
 U 1 1 61D13A27
-P 10050 2000
+P 10600 1650
 AR Path="/607F2E3B/61D13A27" Ref="#PWR0322"  Part="1"
 AR Path="/608AF770/61D13A27" Ref="#PWR?"  Part="1"
-F 0 "#PWR0322" H 10050 1850 50  0001 C CNN
-F 1 "+3.3V" H 10050 2150 50  0000 C CNN
-F 2 "" H 10050 2000 50  0001 C CNN
-F 3 "" H 10050 2000 50  0001 C CNN
-	1    10050 2000
-	1    0    0    -1
-$EndComp
-Wire Wire Line
-	10050 2000 10050 2100
-$Comp
-L Transistor_FET:AO3401A Q301
-U 1 1 61D4997A
-P 10150 2300
-F 0 "Q301" H 10355 2254 50  0000 L CNN
-F 1 "AO3401A" H 10355 2345 50  0000 L CNN
-F 2 "Package_TO_SOT_SMD:SOT-23" H 10350 2225 50  0001 L CIN
-F 3 "http://www.aosmd.com/pdfs/datasheet/AO3401A.pdf" H 10150 2300 50  0001 L CNN
-	1    10150 2300
-	-1   0    0    1
-$EndComp
-Wire Wire Line
-	10350 2300 10500 2300
+F 0 "#PWR0322" H 10600 1500 50  0001 C CNN
+F 1 "+3.3V" H 10600 1800 50  0000 C CNN
+F 2 "" H 10600 1650 50  0001 C CNN
+F 3 "" H 10600 1650 50  0001 C CNN
+	1    10600 1650
+	1    0    0    -1
+$EndComp
 $Comp
 L Device:R_Small R320
 U 1 1 61D8A3A7
-P 10500 2500
+P 10150 2150
 AR Path="/607F2E3B/61D8A3A7" Ref="R320"  Part="1"
 AR Path="/608AF770/61D8A3A7" Ref="R?"  Part="1"
-F 0 "R320" H 10400 2450 50  0000 C CNN
-F 1 "10k" H 10400 2550 50  0000 C CNN
-F 2 "Resistor_SMD:R_0402_1005Metric_Pad0.72x0.64mm_HandSolder" H 10500 2500 50  0001 C CNN
-F 3 "~" H 10500 2500 50  0001 C CNN
-F 4 "C25744" H 10500 2500 50  0001 C CNN "LCSC Part #"
-	1    10500 2500
-	-1   0    0    1
-$EndComp
-$Comp
-L power:GND #PWR0323
-U 1 1 61D8A3AD
-P 10500 2600
-AR Path="/607F2E3B/61D8A3AD" Ref="#PWR0323"  Part="1"
-AR Path="/608AF770/61D8A3AD" Ref="#PWR?"  Part="1"
-F 0 "#PWR0323" H 10500 2350 50  0001 C CNN
-F 1 "GND" H 10505 2427 50  0000 C CNN
-F 2 "" H 10500 2600 50  0001 C CNN
-F 3 "" H 10500 2600 50  0001 C CNN
-	1    10500 2600
-	1    0    0    -1
-$EndComp
-Wire Wire Line
-	10500 2400 10500 2300
-Connection ~ 10500 2300
-Wire Wire Line
-	10500 2300 10750 2300
+F 0 "R320" H 10050 2100 50  0000 C CNN
+F 1 "10k" H 10050 2200 50  0000 C CNN
+F 2 "Resistor_SMD:R_0402_1005Metric_Pad0.72x0.64mm_HandSolder" H 10150 2150 50  0001 C CNN
+F 3 "~" H 10150 2150 50  0001 C CNN
+F 4 "C25744" H 10150 2150 50  0001 C CNN "LCSC Part #"
+	1    10150 2150
+	1    0    0    -1
+$EndComp
 Text Notes 9600 1600 0    50   ~ 0
 USB enabling
+Wire Wire Line
+	10600 1900 10600 2050
+Wire Wire Line
+	10650 2050 10600 2050
+Connection ~ 10600 2050
+Wire Wire Line
+	10600 2050 10600 2150
+Wire Wire Line
+	10000 2350 10150 2350
+Wire Wire Line
+	10150 2350 10150 2250
+Connection ~ 10150 2350
+Wire Wire Line
+	10150 2350 10300 2350
+Wire Wire Line
+	10150 2050 10150 1650
+Wire Wire Line
+	10150 1650 10600 1650
+Connection ~ 10600 1650
+$Comp
+L power:GND #PWR0103
+U 1 1 61DA05DE
+P 10600 2600
+AR Path="/607F2E3B/61DA05DE" Ref="#PWR0103"  Part="1"
+AR Path="/608AF770/61DA05DE" Ref="#PWR?"  Part="1"
+F 0 "#PWR0103" H 10600 2350 50  0001 C CNN
+F 1 "GND" H 10605 2427 50  0000 C CNN
+F 2 "" H 10600 2600 50  0001 C CNN
+F 3 "" H 10600 2600 50  0001 C CNN
+	1    10600 2600
+	1    0    0    -1
+$EndComp
+Wire Wire Line
+	10600 2600 10600 2550
+$Comp
+L Transistor_FET:BSS123 Q301
+U 1 1 61DB8BBC
+P 10500 2350
+F 0 "Q301" H 10704 2396 50  0000 L CNN
+F 1 "BSS123" H 10704 2305 50  0000 L CNN
+F 2 "Package_TO_SOT_SMD:SOT-23" H 10700 2275 50  0001 L CIN
+F 3 "http://www.diodes.com/assets/Datasheets/ds30366.pdf" H 10500 2350 50  0001 L CNN
+	1    10500 2350
+	1    0    0    -1
+$EndComp
 $EndSCHEMATC

Commit message: added files to product pcb
Parts:
- Q301: LCSC Part # (none) -> C431506
- R317: LCSC Part # C25744 -> C25900
Changed lines of the file:
@@
 F 2 "Resistor_SMD:R_0402_1005Metric_Pad0.72x0.64mm_HandSolder" H 9050 4450 50  0001 C CNN
 F 3 "~" H 9050 4450 50  0001 C CNN
-F 4 "C25744" H 9050 4450 50  0001 C CNN "LCSC Part #"
+F 4 "C25900" H 9050 4450 50  0001 C CNN "LCSC Part #"
 	1    9050 4450
 	-1   0    0    1
@@
 F 2 "Package_TO_SOT_SMD:SOT-23" H 10700 2275 50  0001 L CIN
 F 3 "http://www.diodes.com/assets/Datasheets/ds30366.pdf" H 10500 2350 50  0001 L CNN
+F 4 "C431506" H 10500 2350 50  0001 C CNN "LCSC Part #"
 	1    10500 2350
 	1    0    0    -1

Commit message: Changed Crystals
Parts:
- C301: value 4u7 -> 4.7uF; Mouser (none) -> 581-0603ZD475KAT2A
- C302, C303, C304, C305, C308: value 100n -> 0.1uF; Mouser (none) -> 581-0402YD104K
- C306: value 1u -> 1uF; Mouser (none) -> 581-0402YD105KAT4A
- C307: value 10n -> 0.01uF; Mouser (none) -> 581-0402ZC103KAT2A
- C309, C311: value 12p -> 24pF; LCSC Part # C1547 -> (none); Mouser (none) -> 04025U240FAT2A
- C310, C312: value 6.8p -> 13pF; LCSC Part # C1576 -> (none); Mouser (none) -> 581-04023U130FAT2A
- D301: Mouser (none) -> 710-150060BS55040
- L301: value 39n -> 39nH; Mouser (none) -> 710-7447840139
- Q301: Mouser (none) -> 726-BSS123NH6327
- R301, R302: value 2k2 -> 2.2kΩ
- R303, R304, R306, R308, R309, R310, R313, R314: value 100k -> 100kΩ
- R305: value 1k5 -> 787Ω; LCSC Part # C25867 -> (none)
- R307: value 7.5k -> 36kΩ
- R311, R319: value 1k5 -> 1.5kΩ
- R312: value 100 -> 100kΩ
- R315, R316, R318, R320: value 10k -> 10kΩ
- R317: value 4k7 -> 4.7kΩ
- U301: Mouser (none) -> 454-W25Q128JVSIQTR
- U302: Mouser (none) -> 511-STM32F103C8T6
- Y301: value 8Mhz -> 8MHz; footprint Crystal:Crystal_SMD_5032-2Pin_5.0x3.2mm_HandSoldering -> Crystal:Crystal_SMD_HC49-SD_HandSoldering; LCSC Part # C115962 -> (none); Mouser (none) -> 815-ABLS-8.0M-T; Name X50328MSB2GI -> (none)
- Y302: value 32.768KHZ -> 32.768KHz; footprint Crystal:Crystal_SMD_3215-2Pin_3.2x1.5mm -> Crystal:Crystal_SMD_Abracon_ABS25-4Pin_8.0x3.8mm; LCSC Part # C97604 -> (none); Mouser (none) -> 815-ABS25-32.7K-4-T
Other:
- note added: "CLoad = 2 * (CL - Cstray[6pF])\n\nR ext = 1 / (2 * (2 π F[Hz] CLoad[F])"

Commit message: Change part number
Parts:
- Q301: value BSS123 -> SI2312BDS-T1-BE3; footprint Package_TO_SOT_SMD:SOT-23 -> Package_TO_SOT_SMD:SOT-23_Handsoldering; Mouser 726-BSS123NH6327 -> 78-SI2312BDS-T1-BE3
- R301, R302: Mouser (none) -> 652-CR0402FX-2201GLF
- R303, R304, R306, R308, R309, R310, R313, R314: Mouser (none) -> 652-CR0402JW-104GLF
- R305: Mouser (none) -> 652-CR0402-FX7870GLF
- R307: Mouser (none) -> 71-CRCW0402J-36K-E3
- R311: Mouser (none) -> 755-KTR03EZPJ152
- R312: Mouser (none) -> 652-CR0603-FX-103ELF
- R315, R316, R318, R320: LCSC Part # C25744 -> (none); Mouser (none) -> 71-CRCW040210K0FKEDC
- R317: Mouser (none) -> 71-CRCW04024K70FKEDC
- R319: Mouser (none) -> 652-CR0402FX-1501GLF
Changed lines of the file:
@@
 F 2 "Resistor_SMD:R_0402_1005Metric_Pad0.72x0.64mm_HandSolder" H 9050 4850 50  0001 C CNN
 F 3 "~" H 9050 4850 50  0001 C CNN
-F 4 "C25744" H 9050 4850 50  0001 C CNN "LCSC Part #"
+F 4 "" H 9050 4850 50  0001 C CNN "LCSC Part #"
+F 5 "71-CRCW040210K0FKEDC" H 9050 4850 50  0001 C CNN "Mouser"
 	1    9050 4850
 	-1   0    0    1
@@
 F 3 "~" H 5350 4650 50  0001 C CNN
 F 4 "" H 5350 4650 50  0001 C CNN "LCSC Part #"
+F 5 "652-CR0402-FX7870GLF" H 5350 4650 50  0001 C CNN "Mouser"
 	1    5350 4650
 	-1   0    0    1
@@
 F 3 "~" H 6100 6900 50  0001 C CNN
 F 4 "C25918" H 6100 6900 50  0001 C CNN "LCSC Part #"
+F 5 "71-CRCW0402J-36K-E3" H 6100 6900 50  0001 C CNN "Mouser"
 	1    6100 6900
 	-1   0    0    1
@@
 F 3 "~" H 7550 4500 50  0001 C CNN
 F 4 "C22843" H 7550 4500 50  0001 C CNN "LCSC Part #"
+F 5 "755-KTR03EZPJ152" H 7550 4500 50  0001 C CNN "Mouser"
 	1    7550 4500
 	-1   0    0    1
@@
 F 3 "~" H 4250 2650 50  0001 C CNN
 F 4 "C25879" H 4250 2650 50  0001 C CNN "LCSC Part #"
+F 5 "652-CR0402FX-2201GLF" H 4250 2650 50  0001 C CNN "Mouser"
 	1    4250 2650
 	-1   0    0    1
@@
 F 3 "~" H 4050 2650 50  0001 C CNN
 F 4 "C25879" H 4050 2650 50  0001 C CNN "LCSC Part #"
+F 5 "652-CR0402FX-2201GLF" H 4050 2650 50  0001 C CNN "Mouser"
 	1    4050 2650
 	-1   0    0    1
@@
 F 3 "~" H 5350 2650 50  0001 C CNN
 F 4 "C25741" H 5350 2650 50  0001 C CNN "LCSC Part #"
+F 5 "652-CR0402JW-104GLF" H 5350 2650 50  0001 C CNN "Mouser"
 	1    5350 2650
 	-1   0    0    1
@@
 F 3 "~" H 5050 2650 50  0001 C CNN
 F 4 "C25741" H 5050 2650 50  0001 C CNN "LCSC Part #"
+F 5 "652-CR0402JW-104GLF" H 5050 2650 50  0001 C CNN "Mouser"
 	1    5050 2650
 	-1   0    0    1
@@
 F 3 "~" H 8350 2650 50  0001 C CNN
 F 4 "C25741" H 8350 2650 50  0001 C CNN "LCSC Part #"
+F 5 "652-CR0402JW-104GLF" H 8350 2650 50  0001 C CNN "Mouser"
 	1    8350 2650
 	-1   0    0    1
@@
 F 3 "~" H 8050 2650 50  0001 C CNN
 F 4 "C25741" H 8050 2650 50  0001 C CNN "LCSC Part #"
+F 5 "652-CR0402JW-104GLF" H 8050 2650 50  0001 C CNN "Mouser"
 	1    8050 2650
 	-1   0    0    1
@@
 F 2 "Resistor_SMD:R_0402_1005Metric_Pad0.72x0.64mm_HandSolder" H 8950 2650 50  0001 C CNN
 F 3 "~" H 8950 2650 50  0001 C CNN
-F 4 "C25744" H 8950 2650 50  0001 C CNN "LCSC Part #"
+F 4 "" H 8950 2650 50  0001 C CNN "LCSC Part #"
+F 5 "71-CRCW040210K0FKEDC" H 8950 2650 50  0001 C CNN "Mouser"
 	1    8950 2650
 	-1   0    0    1
@@
 F 2 "Resistor_SMD:R_0402_1005Metric_Pad0.72x0.64mm_HandSolder" H 8650 2650 50  0001 C CNN
 F 3 "~" H 8650 2650 50  0001 C CNN
-F 4 "C25744" H 8650 2650 50  0001 C CNN "LCSC Part #"
+F 4 "" H 8650 2650 50  0001 C CNN "LCSC Part #"
+F 5 "71-CRCW040210K0FKEDC" H 8650 2650 50  0001 C CNN "Mouser"
 	1    8650 2650
 	-1   0    0    1
@@
 F 3 "~" H 6050 2650 50  0001 C CNN
 F 4 "C25741" H 6050 2650 50  0001 C CNN "LCSC Part #"
+F 5 "652-CR0402JW-104GLF" H 6050 2650 50  0001 C CNN "Mouser"
 	1    6050 2650
 	-1   0    0    1
@@
 F 3 "~" H 6350 2650 50  0001 C CNN
 F 4 "C25741" H 6350 2650 50  0001 C CNN "LCSC Part #"
+F 5 "652-CR0402JW-104GLF" H 6350 2650 50  0001 C CNN "Mouser"
 	1    6350 2650
 	-1   0    0    1
@@
 F 3 "~" H 7050 2650 50  0001 C CNN
 F 4 "C25741" H 7050 2650 50  0001 C CNN "LCSC Part #"
+F 5 "652-CR0402JW-104GLF" H 7050 2650 50  0001 C CNN "Mouser"
 	1    7050 2650
 	-1   0    0    1
@@
 F 3 "~" H 7350 2650 50  0001 C CNN
 F 4 "C25741" H 7350 2650 50  0001 C CNN "LCSC Part #"
+F 5 "652-CR0402JW-104GLF" H 7350 2650 50  0001 C CNN "Mouser"
 	1    7350 2650
 	-1   0    0    1
@@
 F 3 "~" H 10600 1800 50  0001 C CNN
 F 4 "C25867" H 10600 1800 50  0001 C CNN "LCSC Part #"
+F 5 "652-CR0402FX-1501GLF" H 10600 1800 50  0001 C CNN "Mouser"
 	1    10600 1800
 	-1   0    0    1
@@
 F 3 "~" H 7750 5900 50  0001 C CNN
 F 4 "C25076" H 7750 5900 50  0001 C CNN "LCSC Part #"
+F 5 "652-CR0603-FX-103ELF" H 7750 5900 50  0001 C CNN "Mouser"
 	1    7750 5900
 	-1   0    0    1
@@
 F 3 "~" H 9050 4450 50  0001 C CNN
 F 4 "C25900" H 9050 4450 50  0001 C CNN "LCSC Part #"
+F 5 "71-CRCW04024K70FKEDC" H 9050 4450 50  0001 C CNN "Mouser"
 	1    9050 4450
 	-1   0    0    1
@@
 F 2 "Resistor_SMD:R_0402_1005Metric_Pad0.72x0.64mm_HandSolder" H 10150 2150 50  0001 C CNN
 F 3 "~" H 10150 2150 50  0001 C CNN
-F 4 "C25744" H 10150 2150 50  0001 C CNN "LCSC Part #"
+F 4 "" H 10150 2150 50  0001 C CNN "LCSC Part #"
+F 5 "71-CRCW040210K0FKEDC" H 10150 2150 50  0001 C CNN "Mouser"
 	1    10150 2150
 	1    0    0    -1
@@
 P 10500 2350
 F 0 "Q301" H 10704 2396 50  0000 L CNN
-F 1 "BSS123" H 10704 2305 50  0000 L CNN
-F 2 "Package_TO_SOT_SMD:SOT-23" H 10700 2275 50  0001 L CIN
+F 1 "SI2312BDS-T1-BE3" H 10704 2305 50  0000 L CNN
+F 2 "Package_TO_SOT_SMD:SOT-23_Handsoldering" H 10700 2275 50  0001 L CIN
 F 3 "http://www.diodes.com/assets/Datasheets/ds30366.pdf" H 10500 2350 50  0001 L CNN
 F 4 "C431506" H 10500 2350 50  0001 C CNN "LCSC Part #"
-F 5 "726-BSS123NH6327" H 10500 2350 50  0001 C CNN "Mouser"
+F 5 "78-SI2312BDS-T1-BE3" H 10500 2350 50  0001 C CNN "Mouser"
 	1    10500 2350
 	1    0    0    -1

Commit message: Added descriptions
Parts:
- C309, C311: Mouser 04025U240FAT2A -> 581-04025U240FAT2A
Changed lines of the file:
@@
 F 3 "~" H 4400 4950 50  0001 C CNN
 F 4 "" H 4400 4950 50  0001 C CNN "LCSC Part #"
-F 5 "04025U240FAT2A" H 4400 4950 50  0001 C CNN "Mouser"
+F 5 "581-04025U240FAT2A" H 4400 4950 50  0001 C CNN "Mouser"
 	1    4400 4950
 	1    0    0    -1
@@
 F 3 "~" H 5350 4950 50  0001 C CNN
 F 4 "" H 5350 4950 50  0001 C CNN "LCSC Part #"
-F 5 "04025U240FAT2A" H 5350 4950 50  0001 C CNN "Mouser"
+F 5 "581-04025U240FAT2A" H 5350 4950 50  0001 C CNN "Mouser"
 	1    5350 4950
 	1    0    0    -1
