File: Board_STM32F103C8T6/STM32F103C8T6/PROBES.sch (KiCad schematic (older format))
At the start: 13 parts, among them U701 TLP627

Commit message: Updated board design
work in progress
Parts:
- added C701: 10u, Capacitor_SMD:C_1206_3216Metric_Pad1.33x1.80mm_HandSolder, symbol Device:C_Small
- C702: footprint Capacitor_SMD:C_0603_1608Metric_Pad1.08x0.95mm_HandSolder -> Capacitor_SMD:C_1210_3225Metric_Pad1.33x2.70mm_HandSolder
- C703: renamed from C701; footprint Capacitor_SMD:C_0603_1608Metric_Pad1.08x0.95mm_HandSolder -> Capacitor_SMD:C_1206_3216Metric_Pad1.33x1.80mm_HandSolder
- R701, R702, R706: footprint Resistor_SMD:R_0603_1608Metric_Pad0.98x0.95mm_HandSolder -> Resistor_SMD:R_1206_3216Metric_Pad1.30x1.75mm_HandSolder
- R703, R704, R705: footprint Resistor_SMD:R_0603_1608Metric_Pad0.98x0.95mm_HandSolder -> Resistor_SMD:R_1210_3225Metric_Pad1.30x2.65mm_HandSolder
Connections:
- wire segments 31 -> 36
Changed lines of the file:
@@
 F 0 "R703" V 2254 4000 50  0000 C CNN
 F 1 "4,7K" V 2345 4000 50  0000 C CNN
-F 2 "Resistor_SMD:R_0603_1608Metric_Pad0.98x0.95mm_HandSolder" H 2450 4000 50  0001 C CNN
+F 2 "Resistor_SMD:R_1210_3225Metric_Pad1.30x2.65mm_HandSolder" H 2450 4000 50  0001 C CNN
 F 3 "~" H 2450 4000 50  0001 C CNN
 F 4 "C25804" H 2450 4000 50  0001 C CNN "LCSC Part #"
@@
 F 0 "R704" H 2659 4196 50  0000 L CNN
 F 1 "10K" H 2659 4105 50  0000 L CNN
-F 2 "Resistor_SMD:R_0603_1608Metric_Pad0.98x0.95mm_HandSolder" H 2600 4150 50  0001 C CNN
+F 2 "Resistor_SMD:R_1210_3225Metric_Pad1.30x2.65mm_HandSolder" H 2600 4150 50  0001 C CNN
 F 3 "~" H 2600 4150 50  0001 C CNN
 F 4 "C25804" H 2600 4150 50  0001 C CNN "LCSC Part #"
@@
 F 0 "C702" H 3042 4196 50  0000 L CNN
 F 1 "250n" H 3042 4105 50  0000 L CNN
-F 2 "Capacitor_SMD:C_0603_1608Metric_Pad1.08x0.95mm_HandSolder" H 2950 4150 50  0001 C CNN
+F 2 "Capacitor_SMD:C_1210_3225Metric_Pad1.33x2.70mm_HandSolder" H 2950 4150 50  0001 C CNN
 F 3 "~" H 2950 4150 50  0001 C CNN
 F 4 "C14663" H 2950 4150 50  0001 C CNN "LCSC Part #"
@@
 F 0 "R705" V 3554 4000 50  0000 C CNN
 F 1 "100" V 3645 4000 50  0000 C CNN
-F 2 "Resistor_SMD:R_0603_1608Metric_Pad0.98x0.95mm_HandSolder" H 3750 4000 50  0001 C CNN
+F 2 "Resistor_SMD:R_1210_3225Metric_Pad1.30x2.65mm_HandSolder" H 3750 4000 50  0001 C CNN
 F 3 "~" H 3750 4000 50  0001 C CNN
 F 4 "C22775" H 3750 4000 50  0001 C CNN "LCSC Part #"
@@
 F 0 "R706" H 4959 3946 50  0000 L CNN
 F 1 "10K" H 4959 3855 50  0000 L CNN
-F 2 "Resistor_SMD:R_0603_1608Metric_Pad0.98x0.95mm_HandSolder" H 4900 3900 50  0001 C CNN
+F 2 "Resistor_SMD:R_1206_3216Metric_Pad1.30x1.75mm_HandSolder" H 4900 3900 50  0001 C CNN
 F 3 "~" H 4900 3900 50  0001 C CNN
 F 4 "C25804" H 4900 3900 50  0001 C CNN "LCSC Part #"
@@
 P 2050 5350
 AR Path="/608B029C/608683D4" Ref="C?"  Part="1"
-AR Path="/608D8494/608683D4" Ref="C701"  Part="1"
-F 0 "C701" H 2142 5396 50  0000 L CNN
+AR Path="/608D8494/608683D4" Ref="C703"  Part="1"
+F 0 "C703" H 2142 5396 50  0000 L CNN
 F 1 "10u" H 2142 5305 50  0000 L CNN
-F 2 "Capacitor_SMD:C_0603_1608Metric_Pad1.08x0.95mm_HandSolder" H 2050 5350 50  0001 C CNN
+F 2 "Capacitor_SMD:C_1206_3216Metric_Pad1.33x1.80mm_HandSolder" H 2050 5350 50  0001 C CNN
 F 3 "~" H 2050 5350 50  0001 C CNN
 F 4 "C14663" H 2050 5350 50  0001 C CNN "LCSC Part #"
@@
 F 0 "R701" H 1609 5396 50  0000 L CNN
 F 1 "10K" H 1609 5305 50  0000 L CNN
-F 2 "Resistor_SMD:R_0603_1608Metric_Pad0.98x0.95mm_HandSolder" H 1550 5350 50  0001 C CNN
+F 2 "Resistor_SMD:R_1206_3216Metric_Pad1.30x1.75mm_HandSolder" H 1550 5350 50  0001 C CNN
 F 3 "~" H 1550 5350 50  0001 C CNN
 F 4 "C25804" H 1550 5350 50  0001 C CNN "LCSC Part #"
@@
 F 0 "R702" H 2159 2646 50  0000 L CNN
 F 1 "10K" H 2159 2555 50  0000 L CNN
-F 2 "Resistor_SMD:R_0603_1608Metric_Pad0.98x0.95mm_HandSolder" H 2100 2600 50  0001 C CNN
+F 2 "Resistor_SMD:R_1206_3216Metric_Pad1.30x1.75mm_HandSolder" H 2100 2600 50  0001 C CNN
 F 3 "~" H 2100 2600 50  0001 C CNN
 F 4 "C25804" H 2100 2600 50  0001 C CNN "LCSC Part #"
@@
 L power:+3.3V #PWR0704
 U 1 1 608D87B1
-P 2100 2500
-F 0 "#PWR0704" H 2100 2350 50  0001 C CNN
-F 1 "+3.3V" H 2115 2673 50  0000 C CNN
-F 2 "" H 2100 2500 50  0001 C CNN
-F 3 "" H 2100 2500 50  0001 C CNN
-	1    2100 2500
-	1    0    0    -1
-$EndComp
+P 2100 2350
+F 0 "#PWR0704" H 2100 2200 50  0001 C CNN
+F 1 "+3.3V" H 2115 2523 50  0000 C CNN
+F 2 "" H 2100 2350 50  0001 C CNN
+F 3 "" H 2100 2350 50  0001 C CNN
+	1    2100 2350
+	1    0    0    -1
+$EndComp
+$Comp
+L Device:C_Small C701
+U 1 1 61DBD2BE
+P 2550 2600
+F 0 "C701" H 2642 2646 50  0000 L CNN
+F 1 "10u" H 2642 2555 50  0000 L CNN
+F 2 "Capacitor_SMD:C_1206_3216Metric_Pad1.33x1.80mm_HandSolder" H 2550 2600 50  0001 C CNN
+F 3 "~" H 2550 2600 50  0001 C CNN
+F 4 "C14663" H 2550 2600 50  0001 C CNN "LCSC Part #"
+	1    2550 2600
+	1    0    0    -1
+$EndComp
+$Comp
+L power:GND #PWR0101
+U 1 1 61DBD90C
+P 2550 2800
+F 0 "#PWR0101" H 2550 2550 50  0001 C CNN
+F 1 "GND" H 2555 2627 50  0000 C CNN
+F 2 "" H 2550 2800 50  0001 C CNN
+F 3 "" H 2550 2800 50  0001 C CNN
+	1    2550 2800
+	1    0    0    -1
+$EndComp
+Wire Wire Line
+	2550 2800 2550 2700
+Wire Wire Line
+	2100 2500 2100 2450
+Wire Wire Line
+	2550 2500 2550 2450
+Wire Wire Line
+	2550 2450 2100 2450
+Connection ~ 2100 2450
+Wire Wire Line
+	2100 2450 2100 2350
 $EndSCHEMATC

Commit message: added files to product pcb
Parts:
- C701, C703: LCSC Part # C14663 -> C13585
- C702: value 250n -> 220n; LCSC Part # C14663 -> C396814
- R701, R702, R706: LCSC Part # C25804 -> C17902
- R703: value 4,7K -> 4k7; LCSC Part # C25804 -> C52443
- R704: LCSC Part # C25804 -> C25672
- R705: LCSC Part # C22775 -> C56239
Changed lines of the file:
@@
 P 2450 4000
 F 0 "R703" V 2254 4000 50  0000 C CNN
-F 1 "4,7K" V 2345 4000 50  0000 C CNN
+F 1 "4k7" V 2345 4000 50  0000 C CNN
 F 2 "Resistor_SMD:R_1210_3225Metric_Pad1.30x2.65mm_HandSolder" H 2450 4000 50  0001 C CNN
 F 3 "~" H 2450 4000 50  0001 C CNN
-F 4 "C25804" H 2450 4000 50  0001 C CNN "LCSC Part #"
+F 4 "C52443" H 2450 4000 50  0001 C CNN "LCSC Part #"
 	1    2450 4000
 	0    1    1    0
@@
 F 2 "Resistor_SMD:R_1210_3225Metric_Pad1.30x2.65mm_HandSolder" H 2600 4150 50  0001 C CNN
 F 3 "~" H 2600 4150 50  0001 C CNN
-F 4 "C25804" H 2600 4150 50  0001 C CNN "LCSC Part #"
+F 4 "C25672" H 2600 4150 50  0001 C CNN "LCSC Part #"
 	1    2600 4150
 	1    0    0    -1
@@
 P 2950 4150
 F 0 "C702" H 3042 4196 50  0000 L CNN
-F 1 "250n" H 3042 4105 50  0000 L CNN
+F 1 "220n" H 3042 4105 50  0000 L CNN
 F 2 "Capacitor_SMD:C_1210_3225Metric_Pad1.33x2.70mm_HandSolder" H 2950 4150 50  0001 C CNN
 F 3 "~" H 2950 4150 50  0001 C CNN
-F 4 "C14663" H 2950 4150 50  0001 C CNN "LCSC Part #"
+F 4 "C396814" H 2950 4150 50  0001 C CNN "LCSC Part #"
 	1    2950 4150
 	1    0    0    -1
@@
 F 2 "Resistor_SMD:R_1210_3225Metric_Pad1.30x2.65mm_HandSolder" H 3750 4000 50  0001 C CNN
 F 3 "~" H 3750 4000 50  0001 C CNN
-F 4 "C22775" H 3750 4000 50  0001 C CNN "LCSC Part #"
+F 4 "C56239" H 3750 4000 50  0001 C CNN "LCSC Part #"
 	1    3750 4000
 	0    1    1    0
@@
 F 2 "Resistor_SMD:R_1206_3216Metric_Pad1.30x1.75mm_HandSolder" H 4900 3900 50  0001 C CNN
 F 3 "~" H 4900 3900 50  0001 C CNN
-F 4 "C25804" H 4900 3900 50  0001 C CNN "LCSC Part #"
+F 4 "C17902" H 4900 3900 50  0001 C CNN "LCSC Part #"
 	1    4900 3900
 	1    0    0    -1
@@
 F 2 "Capacitor_SMD:C_1206_3216Metric_Pad1.33x1.80mm_HandSolder" H 2050 5350 50  0001 C CNN
 F 3 "~" H 2050 5350 50  0001 C CNN
-F 4 "C14663" H 2050 5350 50  0001 C CNN "LCSC Part #"
+F 4 "C13585" H 2050 5350 50  0001 C CNN "LCSC Part #"
 	1    2050 5350
 	1    0    0    -1
@@
 F 2 "Resistor_SMD:R_1206_3216Metric_Pad1.30x1.75mm_HandSolder" H 1550 5350 50  0001 C CNN
 F 3 "~" H 1550 5350 50  0001 C CNN
-F 4 "C25804" H 1550 5350 50  0001 C CNN "LCSC Part #"
+F 4 "C17902" H 1550 5350 50  0001 C CNN "LCSC Part #"
 	1    1550 5350
 	1    0    0    -1
@@
 F 2 "Resistor_SMD:R_1206_3216Metric_Pad1.30x1.75mm_HandSolder" H 2100 2600 50  0001 C CNN
 F 3 "~" H 2100 2600 50  0001 C CNN
-F 4 "C25804" H 2100 2600 50  0001 C CNN "LCSC Part #"
+F 4 "C17902" H 2100 2600 50  0001 C CNN "LCSC Part #"
 	1    2100 2600
 	1    0    0    -1
@@
 F 2 "Capacitor_SMD:C_1206_3216Metric_Pad1.33x1.80mm_HandSolder" H 2550 2600 50  0001 C CNN
 F 3 "~" H 2550 2600 50  0001 C CNN
-F 4 "C14663" H 2550 2600 50  0001 C CNN "LCSC Part #"
+F 4 "C13585" H 2550 2600 50  0001 C CNN "LCSC Part #"
 	1    2550 2600
 	1    0    0    -1

Commit message: Changed Crystals
Parts:
- C701, C703: value 10u -> 10uF; Mouser (none) -> 581-1206DD106KAT2A
- C702: value 220n -> 0.1uF; Mouser (none) -> 581-1210VC224KAT2A
- D703: Mouser (none) -> 78-1N4148WS-E3-18
- D704: Mouser (none) -> 78-BZT52C5V1-E3-18
- R701, R702, R704, R706: value 10K -> 10kΩ
- R703: value 4k7 -> 10kΩ
- R705: value 100 -> 100kΩ
Changed lines of the file:
@@
 P 2450 4000
 F 0 "R703" V 2254 4000 50  0000 C CNN
-F 1 "4k7" V 2345 4000 50  0000 C CNN
+F 1 "10kΩ" V 2345 4000 50  0000 C CNN
 F 2 "Resistor_SMD:R_1210_3225Metric_Pad1.30x2.65mm_HandSolder" H 2450 4000 50  0001 C CNN
 F 3 "~" H 2450 4000 50  0001 C CNN
@@
 P 2600 4150
 F 0 "R704" H 2659 4196 50  0000 L CNN
-F 1 "10K" H 2659 4105 50  0000 L CNN
+F 1 "10kΩ" H 2659 4105 50  0000 L CNN
 F 2 "Resistor_SMD:R_1210_3225Metric_Pad1.30x2.65mm_HandSolder" H 2600 4150 50  0001 C CNN
 F 3 "~" H 2600 4150 50  0001 C CNN
@@
 P 2950 4150
 F 0 "C702" H 3042 4196 50  0000 L CNN
-F 1 "220n" H 3042 4105 50  0000 L CNN
+F 1 "0.1uF" H 3042 4105 50  0000 L CNN
 F 2 "Capacitor_SMD:C_1210_3225Metric_Pad1.33x2.70mm_HandSolder" H 2950 4150 50  0001 C CNN
 F 3 "~" H 2950 4150 50  0001 C CNN
 F 4 "C396814" H 2950 4150 50  0001 C CNN "LCSC Part #"
+F 5 "581-1210VC224KAT2A" H 2950 4150 50  0001 C CNN "Mouser"
 	1    2950 4150
 	1    0    0    -1
@@
 F 3 "~" V 3400 4150 50  0001 C CNN
 F 4 "C78479" H 3400 4150 50  0001 C CNN "LCSC Part #"
+F 5 "78-BZT52C5V1-E3-18" H 3400 4150 50  0001 C CNN "Mouser"
 	1    3400 4150
 	0    1    1    0
@@
 F 3 "~" V 3100 4000 50  0001 C CNN
 F 4 "C2128" H 3100 4000 50  0001 C CNN "LCSC Part #"
+F 5 "78-1N4148WS-E3-18" H 3100 4000 50  0001 C CNN "Mouser"
 	1    3100 4000
 	-1   0    0    1
@@
 P 3750 4000
 F 0 "R705" V 3554 4000 50  0000 C CNN
-F 1 "100" V 3645 4000 50  0000 C CNN
+F 1 "100kΩ" V 3645 4000 50  0000 C CNN
 F 2 "Resistor_SMD:R_1210_3225Metric_Pad1.30x2.65mm_HandSolder" H 3750 4000 50  0001 C CNN
 F 3 "~" H 3750 4000 50  0001 C CNN
@@
 P 4900 3900
 F 0 "R706" H 4959 3946 50  0000 L CNN
-F 1 "10K" H 4959 3855 50  0000 L CNN
+F 1 "10kΩ" H 4959 3855 50  0000 L CNN
 F 2 "Resistor_SMD:R_1206_3216Metric_Pad1.30x1.75mm_HandSolder" H 4900 3900 50  0001 C CNN
 F 3 "~" H 4900 3900 50  0001 C CNN
@@
 AR Path="/608D8494/608683D4" Ref="C703"  Part="1"
 F 0 "C703" H 2142 5396 50  0000 L CNN
-F 1 "10u" H 2142 5305 50  0000 L CNN
+F 1 "10uF" H 2142 5305 50  0000 L CNN
 F 2 "Capacitor_SMD:C_1206_3216Metric_Pad1.33x1.80mm_HandSolder" H 2050 5350 50  0001 C CNN
 F 3 "~" H 2050 5350 50  0001 C CNN
 F 4 "C13585" H 2050 5350 50  0001 C CNN "LCSC Part #"
+F 5 "581-1206DD106KAT2A" H 2050 5350 50  0001 C CNN "Mouser"
 	1    2050 5350
 	1    0    0    -1
@@
 P 1550 5350
 F 0 "R701" H 1609 5396 50  0000 L CNN
-F 1 "10K" H 1609 5305 50  0000 L CNN
+F 1 "10kΩ" H 1609 5305 50  0000 L CNN
 F 2 "Resistor_SMD:R_1206_3216Metric_Pad1.30x1.75mm_HandSolder" H 1550 5350 50  0001 C CNN
 F 3 "~" H 1550 5350 50  0001 C CNN
@@
 P 2100 2600
 F 0 "R702" H 2159 2646 50  0000 L CNN
-F 1 "10K" H 2159 2555 50  0000 L CNN
+F 1 "10kΩ" H 2159 2555 50  0000 L CNN
 F 2 "Resistor_SMD:R_1206_3216Metric_Pad1.30x1.75mm_HandSolder" H 2100 2600 50  0001 C CNN
 F 3 "~" H 2100 2600 50  0001 C CNN
@@
 P 2550 2600
 F 0 "C701" H 2642 2646 50  0000 L CNN
-F 1 "10u" H 2642 2555 50  0000 L CNN
+F 1 "10uF" H 2642 2555 50  0000 L CNN
 F 2 "Capacitor_SMD:C_1206_3216Metric_Pad1.33x1.80mm_HandSolder" H 2550 2600 50  0001 C CNN
 F 3 "~" H 2550 2600 50  0001 C CNN
 F 4 "C13585" H 2550 2600 50  0001 C CNN "LCSC Part #"
+F 5 "581-1206DD106KAT2A" H 2550 2600 50  0001 C CNN "Mouser"
 	1    2550 2600
 	1    0    0    -1

Commit message: Change part number
Parts:
- D701, D702: footprint Diode_SMD:D_SMA -> Diode_SMD:D_SMA_Handsoldering
- D703: footprint Diode_SMD:D_SOD-323F -> Diode_SMD:D_SOD-323_HandSoldering; LCSC Part # C2128 -> (none); Mouser 78-1N4148WS-E3-18 -> 241-1N4148WSR100001
- R701, R702, R706: Mouser (none) -> 652-CR1206FX-1002ELF
- R703, R704: Mouser (none) -> 603-RC1210FR-0710KL
- R705: Mouser (none) -> 660-RK73B2ETTD104J
Changed lines of the file:
@@
 F 3 "~" H 2450 4000 50  0001 C CNN
 F 4 "C52443" H 2450 4000 50  0001 C CNN "LCSC Part #"
+F 5 "603-RC1210FR-0710KL" H 2450 4000 50  0001 C CNN "Mouser"
 	1    2450 4000
 	0    1    1    0
@@
 F 3 "~" H 2600 4150 50  0001 C CNN
 F 4 "C25672" H 2600 4150 50  0001 C CNN "LCSC Part #"
+F 5 "603-RC1210FR-0710KL" H 2600 4150 50  0001 C CNN "Mouser"
 	1    2600 4150
 	1    0    0    -1
@@
 F 0 "D702" H 2100 3793 50  0000 C CNN
 F 1 "1N4007F" H 2100 3884 50  0000 C CNN
-F 2 "Diode_SMD:D_SMA" V 2100 4000 50  0001 C CNN
+F 2 "Diode_SMD:D_SMA_Handsoldering" V 2100 4000 50  0001 C CNN
 F 3 "~" V 2100 4000 50  0001 C CNN
 F 4 "C110856" H 2100 4000 50  0001 C CNN "LCSC Part #"
@@
 F 0 "D701" V 1904 4220 50  0000 L CNN
 F 1 "1N4007F" V 1995 4220 50  0000 L CNN
-F 2 "Diode_SMD:D_SMA" V 1950 4150 50  0001 C CNN
+F 2 "Diode_SMD:D_SMA_Handsoldering" V 1950 4150 50  0001 C CNN
 F 3 "~" V 1950 4150 50  0001 C CNN
 F 4 "C110856" H 1950 4150 50  0001 C CNN "LCSC Part #"
@@
 F 0 "D703" H 3100 3793 50  0000 C CNN
 F 1 "1N4148WS" H 3100 3884 50  0000 C CNN
-F 2 "Diode_SMD:D_SOD-323F" V 3100 4000 50  0001 C CNN
+F 2 "Diode_SMD:D_SOD-323_HandSoldering" V 3100 4000 50  0001 C CNN
 F 3 "~" V 3100 4000 50  0001 C CNN
-F 4 "C2128" H 3100 4000 50  0001 C CNN "LCSC Part #"
-F 5 "78-1N4148WS-E3-18" H 3100 4000 50  0001 C CNN "Mouser"
+F 4 "" H 3100 4000 50  0001 C CNN "LCSC Part #"
+F 5 "241-1N4148WSR100001" H 3100 4000 50  0001 C CNN "Mouser"
 	1    3100 4000
 	-1   0    0    1
@@
 F 3 "~" H 3750 4000 50  0001 C CNN
 F 4 "C56239" H 3750 4000 50  0001 C CNN "LCSC Part #"
+F 5 "660-RK73B2ETTD104J" H 3750 4000 50  0001 C CNN "Mouser"
 	1    3750 4000
 	0    1    1    0
@@
 F 3 "~" H 4900 3900 50  0001 C CNN
 F 4 "C17902" H 4900 3900 50  0001 C CNN "LCSC Part #"
+F 5 "652-CR1206FX-1002ELF" H 4900 3900 50  0001 C CNN "Mouser"
 	1    4900 3900
 	1    0    0    -1
@@
 F 3 "~" H 1550 5350 50  0001 C CNN
 F 4 "C17902" H 1550 5350 50  0001 C CNN "LCSC Part #"
+F 5 "652-CR1206FX-1002ELF" H 1550 5350 50  0001 C CNN "Mouser"
 	1    1550 5350
 	1    0    0    -1
@@
 F 3 "~" H 2100 2600 50  0001 C CNN
 F 4 "C17902" H 2100 2600 50  0001 C CNN "LCSC Part #"
+F 5 "652-CR1206FX-1002ELF" H 2100 2600 50  0001 C CNN "Mouser"
 	1    2100 2600
 	1    0    0    -1

Commit message: Added descriptions
Parts:
- D701, D702: Mouser (none) -> 621-S1B-F
- R705: value 100kΩ -> 100Ω; Mouser 660-RK73B2ETTD104J -> 660-RK73B2ETTD101J
Changed lines of the file:
@@
 F 3 "~" V 2100 4000 50  0001 C CNN
 F 4 "C110856" H 2100 4000 50  0001 C CNN "LCSC Part #"
+F 5 "621-S1B-F" H 2100 4000 50  0001 C CNN "Mouser"
 	1    2100 4000
 	-1   0    0    1
@@
 F 3 "~" V 1950 4150 50  0001 C CNN
 F 4 "C110856" H 1950 4150 50  0001 C CNN "LCSC Part #"
+F 5 "621-S1B-F" H 1950 4150 50  0001 C CNN "Mouser"
 	1    1950 4150
 	0    1    1    0
@@
 P 3750 4000
 F 0 "R705" V 3554 4000 50  0000 C CNN
-F 1 "100kΩ" V 3645 4000 50  0000 C CNN
+F 1 "100Ω" V 3645 4000 50  0000 C CNN
 F 2 "Resistor_SMD:R_1210_3225Metric_Pad1.30x2.65mm_HandSolder" H 3750 4000 50  0001 C CNN
 F 3 "~" H 3750 4000 50  0001 C CNN
 F 4 "C56239" H 3750 4000 50  0001 C CNN "LCSC Part #"
-F 5 "660-RK73B2ETTD104J" H 3750 4000 50  0001 C CNN "Mouser"
+F 5 "660-RK73B2ETTD101J" H 3750 4000 50  0001 C CNN "Mouser"
 	1    3750 4000
 	0    1    1    0

Commit message: Update PROBES.sch
Parts:
- C702: Mouser 581-1210VC224KAT2A -> 80-C1210V104KCR
Changed lines of the file:
@@
 F 3 "~" H 2950 4150 50  0001 C CNN
 F 4 "C396814" H 2950 4150 50  0001 C CNN "LCSC Part #"
-F 5 "581-1210VC224KAT2A" H 2950 4150 50  0001 C CNN "Mouser"
+F 5 "80-C1210V104KCR" H 2950 4150 50  0001 C CNN "Mouser"
 	1    2950 4150
 	1    0    0    -1
